File: boards/power-tp4056-5v-ups/power-tp4056-5v-ups.kicad_pcb (KiCad board)
At the start: 2 copper layers, 52.5 x 22.9 mm, 44 parts, among them J0 USB_C_Receptacle_PowerOnly_6P, J1 USB_C_Receptacle_PowerOnly_6P, J101 Conn_01x01, J102 Conn_01x01, J201 Conn_01x01, J202 Conn_01x01, J301 Conn_01x01, J302 Conn_01x01, Q1 AO3401A, Q2 AO3401A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

Commit message: Remove extra diode, fix silkscreen text on power-tp4056-5v-ups
Parts:
- removed D3: SS34, custom:D_SMA_simple
Other:
- board text added: "TP4056, XB5350D0, MT3608"
- board text removed: "TP4056, XB5350D0, MT3680"
