File: dev-boards/power-18650-holder/power-18650-holder.kicad_pcb (KiCad board)
At the start: 2 copper layers, 82 x 40 mm, 24 parts, among them J1 JST XH/PH, J2 JST XH/PH, J3 Screw_Terminal_01x02, J4 Screw_Terminal_01x02

Commit message: Add missing footprints for power-18650-holder
Parts:
- J3, J4: footprint custom:Conn_Combo_TerminalBlock_P3.5-P5.08_pad2gnd -> custom:Conn_Combo_TerminalBlock_P3.5-P5.08_1x02_pad2gnd
Changed lines of the file:
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@@
 		(at 196.5 48 180)
 		(property "Reference" "J2"
-			(at 0 -4 360)
+			(at 0 -4 0)
 			(layer "F.SilkS")
 			(hide yes)
@@
 		)
 		(property "Value" "JST XH/PH"
-			(at 0 4 360)
+			(at 0 4 0)
 			(layer "F.Fab")
 			(effects
@@
 		)
 		(property "Footprint" "custom:Conn_Combo_JST-1x02-XH_PH-THT-pad2gnd"
-			(at 0 0 360)
+			(at 0 0 0)
 			(layer "F.Fab")
 			(hide yes)
@@
 		)
 		(property "Datasheet" ""
-			(at 0 0 360)
+			(at 0 0 0)
 			(layer "F.Fab")
 			(hide yes)
@@
 		)
 		(property "Description" "Generic connector, single row, 01x02, script generated (kicad-library-utils/schlib/autogen/connector/)"
-			(at 0 0 360)
+			(at 0 0 0)
 			(layer "F.Fab")
 			(hide yes)
@@
 		)
 		(fp_text user "${REFERENCE}"
-			(at 0 0 360)
+			(at 0 0 0)
 			(layer "F.Fab")
 			(effects
@@
 		(at 159.5 44 180)
 		(property "Reference" "G***"
-			(at 0 0 360)
+			(at 0 0 0)
 			(layer "F.SilkS")
 			(hide yes)
@@
 		)
 		(property "Value" "LOGO"
-			(at 0.75 0 360)
+			(at 0.75 0 0)
 			(layer "F.SilkS")
 			(hide yes)
@@
 		)
 		(property "Footprint" "graphics:oshw-logo-3mm"
-			(at 0 0 360)
+			(at 0 0 0)
 			(layer "F.Fab")
 			(hide yes)
@@
 		)
 		(property "Datasheet" ""
-			(at 0 0 360)
+			(at 0 0 0)
 			(layer "F.Fab")
 			(hide yes)
@@
 		)
 		(property "Description" ""
-			(at 0 0 360)
+			(at 0 0 0)
 			(layer "F.Fab")
 			(hide yes)
@@
 		)
 	)
-	(footprint "custom:Conn_Combo_TerminalBlock_P3.5-P5.08_pad2gnd"
+	(footprint "custom:Conn_Combo_TerminalBlock_P3.5-P5.08_1x02_pad2gnd"
 		(layer "F.Cu")
 		(at 146.045 43.945 180)
@@
 		(tags "THT Terminal Block Phoenix MKDS-1,5-2-5.08 pitch 5.08mm size 10.2x9.8mm^2 drill 1.3mm pad 2.6mm")
 		(property "Reference" "J4"
-			(at 2.54 -6.26 360)
+			(at 2.54 -6.26 180)
 			(layer "F.SilkS")
 			(hide yes)
@@
 		)
 		(property "Value" "Screw_Terminal_01x02"
-			(at 2.54 5.66 360)
+			(at 2.54 5.66 180)
 			(layer "F.Fab")
 			(effects
@@
 			)
 		)
-		(property "Footprint" "custom:Conn_Combo_TerminalBlock_P3.5-P5.08_pad2gnd"
+		(property "Footprint" "custom:Conn_Combo_TerminalBlock_P3.5-P5.08_1x02_pad2gnd"
 			(at 0 0 180)
 			(unlocked yes)
@@
 		)
 		(fp_text user "${REFERENCE}"
-			(at 2.54 3.2 360)
+			(at 2.54 3.2 180)
 			(layer "F.Fab")
 			(effects
@@
 		)
 	)
-	(footprint "custom:Conn_Combo_TerminalBlock_P3.5-P5.08_pad2gnd"
+	(footprint "custom:Conn_Combo_TerminalBlock_P3.5-P5.08_1x02_pad2gnd"
 		(layer "F.Cu")
 		(at 194.205 76.305)
@@
 			)
 		)
-		(property "Footprint" "custom:Conn_Combo_TerminalBlock_P3.5-P5.08_pad2gnd"
+		(property "Footprint" "custom:Conn_Combo_TerminalBlock_P3.5-P5.08_1x02_pad2gnd"
 			(at 0 0 0)
 			(unlocked yes)
@@
 				(xy 171 54.5) (xy 192 54.5) (xy 196.5 50) (xy 196.5 47) (xy 199 47) (xy 199 50) (xy 199 54.5) (xy 195 58.5)
 				(xy 195 61.5) (xy 196.5 63) (xy 196.5 78) (xy 193 78) (xy 193 66.5) (xy 187.5 61) (xy 171 61) (xy 170 62)
-				(xy 169 61) (xy 152 61) (xy 149.5 63.5) (xy 149.5 63.5) (xy 143.5 69.5) (xy 143.5 73) (xy 141.5 73)
-				(xy 141.5 69.5) (xy 134.5 62.5) (xy 131 62.5) (xy 131 57.5) (xy 134 57.5) (xy 144 47.5) (xy 144 42.5)
+				(xy 169 61) (xy 152 61) (xy 149.5 63.5) (xy 143.5 69.5) (xy 143.5 73) (xy 141.5 73) (xy 141.5 69.5)
+				(xy 134.5 62.5) (xy 131 62.5) (xy 131 57.5) (xy 134 57.5) (xy 144 47.5) (xy 144 42.5)
 			)
 		)
