File: dev-boards/power-18650-holder/power-18650-holder.kicad_sch (KiCad schematic)
At the start: 9 parts, among them J1 JST XH/PH, J2 JST XH/PH, J3 Screw_Terminal_01x02, J4 Screw_Terminal_01x02

Commit message: Add missing footprints for power-18650-holder
Parts:
- J3, J4: footprint custom:Conn_Combo_TerminalBlock_P3.5-P5.08_pad2gnd -> custom:Conn_Combo_TerminalBlock_P3.5-P5.08_1x02_pad2gnd
Changed lines of the file:
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@@
 			)
 		)
-		(property "Footprint" "custom:Conn_Combo_TerminalBlock_P3.5-P5.08_pad2gnd"
+		(property "Footprint" "custom:Conn_Combo_TerminalBlock_P3.5-P5.08_1x02_pad2gnd"
 			(at 215.9 102.87 0)
 			(effects
@@
 			)
 		)
-		(property "Footprint" "custom:Conn_Combo_TerminalBlock_P3.5-P5.08_pad2gnd"
+		(property "Footprint" "custom:Conn_Combo_TerminalBlock_P3.5-P5.08_1x02_pad2gnd"
 			(at 215.9 90.17 0)
 			(effects
