File: pcb-stackable-v2-dev/lcd-round/lcd-round.kicad_pcb (KiCad board)
At the start: 2 copper layers, 35 x 35 mm, 16 parts, among them J1 JST SH, J2 Pin headers, J3 Pin headers, Q1 BSS138

Commit message: Tweak silkscreen on lcd-round
Parts:
- moved REF** 25.7 mm to (85.8, 69.8)
- moved G*** 25.3 mm to (114.0, 69.8)
Other:
- board text added: "rev 1"
