File: dev/stackable2/esp-neopixel-driver/esp-neopixel-driver.kicad_sch (KiCad schematic)
At the start: 43 parts, among them J1 STEMMA-Signal, J2 STEMMA-Signal, J3 Qwiic, J4 Qwiic, J7 Barrel_Jack_Switch, Q1 BSS138, Q2 2N7002DW, U1 TPS563201, U2 INA3221, U3 VEML6030

Commit message: Migrate ESP32 module library references in projects
Parts:
- SM1: footprint aliexpress:ESP32-C3-Super-Mini-Castellated-SMD-only -> modules:ESP32-C3-Super-Mini-Castellated-SMD-only; symbol aliexpress:ESP32-C3-Super-Mini -> modules:ESP32-C3-Super-Mini
Changed lines of the file:
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@@
 	)
 	(symbol
-		(lib_id "aliexpress:ESP32-C3-Super-Mini")
+		(lib_id "modules:ESP32-C3-Super-Mini")
 		(at 53.34 39.37 0)
 		(unit 1)
@@
 			)
 		)
-		(property "Footprint" "aliexpress:ESP32-C3-Super-Mini-Castellated-SMD-only"
+		(property "Footprint" "modules:ESP32-C3-Super-Mini-Castellated-SMD-only"
 			(at 53.34 23.622 0)
 			(effects
