File: dev/misc/esp-doorbell-dev/esp-doorbell-dev.kicad_sch (KiCad schematic)
At the start: 26 parts, among them J1 JST XH, J2 Screw_Terminal_01x02, J3 JST XH/PH, J4 JST PH, Q1 BSS84, Q2 BSS84, Q3 BSS84, Q4 2N7002DW, Q5 BSS138, U1 WS2811F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

Commit message: Migrate ESP32 module library references in projects
Parts:
- SM1: footprint aliexpress:ESP32-C3-Super-Mini-Pins -> modules:ESP32-C3-Super-Mini-Pins; symbol aliexpress:ESP32-C3-Super-Mini -> modules:ESP32-C3-Super-Mini
Changed lines of the file:
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@@
 	)
 	(symbol
-		(lib_id "aliexpress:ESP32-C3-Super-Mini")
+		(lib_id "modules:ESP32-C3-Super-Mini")
 		(at 49.53 41.91 0)
 		(unit 1)
@@
 			)
 		)
-		(property "Footprint" "aliexpress:ESP32-C3-Super-Mini-Pins"
+		(property "Footprint" "modules:ESP32-C3-Super-Mini-Pins"
 			(at 49.53 26.162 0)
 			(effects

Commit message: Migrate DFR0299 (DFPlayer Mini)
Parts:
- SM2: footprint aliexpress:DFPlayer-Mini-DFR0299-module -> modules:DFPlayer-Mini-DFR0299-module; symbol aliexpress:DFR0299 -> modules:DFR0299
Changed lines of the file:
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@@
 	)
 	(symbol
-		(lib_id "aliexpress:DFR0299")
+		(lib_id "modules:DFR0299")
 		(at 106.68 162.56 0)
 		(unit 1)
@@
 			)
 		)
-		(property "Footprint" "aliexpress:DFPlayer-Mini-DFR0299-module"
+		(property "Footprint" "modules:DFPlayer-Mini-DFR0299-module"
 			(at 106.68 162.56 0)
 			(effects

Commit message: Migrate G3MB-202P-5VDC solid state relay module
Parts:
- U2: footprint aliexpress:RELAY-G3MB-202P-5VDC -> custom:RELAY-G3MB-202P-5VDC; symbol aliexpress:G3MB-202P-5VDC -> custom:G3MB-202P-5VDC
Changed lines of the file:
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@@
 	)
 	(symbol
-		(lib_id "aliexpress:G3MB-202P-5VDC")
+		(lib_id "custom:G3MB-202P-5VDC")
 		(at 172.72 118.11 0)
 		(unit 1)
@@
 			)
 		)
-		(property "Footprint" "aliexpress:RELAY-G3MB-202P-5VDC"
+		(property "Footprint" "custom:RELAY-G3MB-202P-5VDC"
 			(at 167.64 123.19 0)
 			(effects

Commit message: Migrate 0.96" OLED symbol, footprint, and model to modules
Parts:
- SM5: footprint aliexpress:LCD-OLED-0.96-module-noholes -> modules:LCD-OLED-0.96-module-noholes; symbol aliexpress:OLED-0.96mm-I2C-module -> modules:OLED-0.96mm-I2C-module
Changed lines of the file:
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@@
 	)
 	(symbol
-		(lib_id "aliexpress:OLED-0.96mm-I2C-module")
+		(lib_id "modules:OLED-0.96mm-I2C-module")
 		(at 80.01 114.3 0)
 		(unit 1)
@@
 			)
 		)
-		(property "Footprint" "aliexpress:LCD-OLED-0.96-module-noholes"
+		(property "Footprint" "modules:LCD-OLED-0.96-module-noholes"
 			(at 80.01 125.73 0)
 			(effects
