File: dev/misc/rotary-encoder-module/rotary-encoder-module.kicad_pcb (KiCad board)
At the start: 2 copper layers, 15 x 21.2 mm, 16 parts, among them J1 JST SH, J2 Pin headers, SW1 RotaryEncoder_Switch_MP

Commit message: Migrate JST SH connector footprints from `custom` to `connectors` library
Parts:
- J1: footprint custom:JST_SH_SM05B-SRSS-TB_1x05-1MP_P1.00mm_Horizontal -> connectors:JST_SH_SM05B-SRSS-TB_1x05-1MP_P1.00mm_Horizontal
Changed lines of the file:
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@@
 		)
 	)
-	(footprint "custom:JST_SH_SM05B-SRSS-TB_1x05-1MP_P1.00mm_Horizontal"
+	(footprint "connectors:JST_SH_SM05B-SRSS-TB_1x05-1MP_P1.00mm_Horizontal"
 		(layer "B.Cu")
 		(at 180 106.5 180)
@@
 			)
 		)
-		(property "Footprint" "custom:JST_SH_SM05B-SRSS-TB_1x05-1MP_P1.00mm_Horizontal"
+		(property "Footprint" "connectors:JST_SH_SM05B-SRSS-TB_1x05-1MP_P1.00mm_Horizontal"
 			(at 0 0 0)
 			(unlocked yes)
