File: dev/stackable2/esp-3dp/esp-3dp.kicad_pcb (KiCad board)
At the start: 2 copper layers, 40 x 40 mm, 46 parts, among them J0 Barrel_Jack_Switch, J1 Barrel_Jack_Switch, J2 JST SH, J3 JST SH, J4 JST XH/PH, J5 Qwiic, J6 Pin headers, M1 KF2510, Q1 2N7002DW, Q2 2N7002DW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

Commit message: Migrate ESP32 module library references in projects
Parts:
- SM1: footprint aliexpress:ESP32-C3-Super-Mini-Castellated-SMD-only -> modules:ESP32-C3-Super-Mini-Castellated-SMD-only
Changed lines of the file:
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@@
 		)
 	)
-	(footprint "aliexpress:ESP32-C3-Super-Mini-Castellated-SMD-only"
+	(footprint "modules:ESP32-C3-Super-Mini-Castellated-SMD-only"
 		(layer "B.Cu")
 		(at 100 59.0435 180)
@@
 			)
 		)
-		(property "Footprint" "aliexpress:ESP32-C3-Super-Mini-Castellated-SMD-only"
+		(property "Footprint" "modules:ESP32-C3-Super-Mini-Castellated-SMD-only"
 			(at 0 0 0)
 			(unlocked yes)
@@
 			)
 		)
-		(model "${KIPRJMOD}/libraries/aliexpress.3dshapes/ESP32-C3-SuperMini.step"
+		(model "${KIPRJMOD}/libraries/modules.3dshapes/ESP32-C3-SuperMini.step"
 			(offset
 				(xyz 0 -2.3 0)

Commit message: Migrate JST SH connector footprints from `custom` to `connectors` library
Parts:
- J2, J3: footprint custom:JST_SH_SM05B-SRSS-TB_1x05-1MP_P1.00mm_Horizontal -> connectors:JST_SH_SM05B-SRSS-TB_1x05-1MP_P1.00mm_Horizontal
Changed lines of the file:
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@@
 		)
 	)
-	(footprint "custom:JST_SH_SM05B-SRSS-TB_1x05-1MP_P1.00mm_Horizontal"
+	(footprint "connectors:JST_SH_SM05B-SRSS-TB_1x05-1MP_P1.00mm_Horizontal"
 		(layer "F.Cu")
 		(at 83.5 78.5 -90)
@@
 			)
 		)
-		(property "Footprint" "custom:JST_SH_SM05B-SRSS-TB_1x05-1MP_P1.00mm_Horizontal"
+		(property "Footprint" "connectors:JST_SH_SM05B-SRSS-TB_1x05-1MP_P1.00mm_Horizontal"
 			(at 0 0 -90)
 			(unlocked yes)
@@
 		)
 	)
-	(footprint "custom:JST_SH_SM05B-SRSS-TB_1x05-1MP_P1.00mm_Horizontal"
+	(footprint "connectors:JST_SH_SM05B-SRSS-TB_1x05-1MP_P1.00mm_Horizontal"
 		(layer "F.Cu")
 		(at 116.5 78.5 90)
@@
 			)
 		)
-		(property "Footprint" "custom:JST_SH_SM05B-SRSS-TB_1x05-1MP_P1.00mm_Horizontal"
+		(property "Footprint" "connectors:JST_SH_SM05B-SRSS-TB_1x05-1MP_P1.00mm_Horizontal"
 			(at 0 0 90)
 			(unlocked yes)
