File: dev/stackable2/esp-lcd-dev/esp-lcd-dev.kicad_pcb (KiCad board)
At the start: 2 copper layers, 40 x 40 mm, 39 parts, among them J1 JST XH/PH, J2 Qwiic, J3 Qwiic, J4 STEMMA-Signal, J5 JST SH, J6 Pin headers, J7 Pin headers, J8 Pin headers, Q1 2N7002DW, U1 VEML7700

Commit message: Migrate ESP32 module library references in projects
Parts:
- SM1: footprint aliexpress:ESP32-C3-Super-Mini-Castellated-SMD-only -> modules:ESP32-C3-Super-Mini-Castellated-SMD-only
Changed lines of the file:
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@@
 		)
 	)
-	(footprint "aliexpress:ESP32-C3-Super-Mini-Castellated-SMD-only"
+	(footprint "modules:ESP32-C3-Super-Mini-Castellated-SMD-only"
 		(layer "B.Cu")
 		(at 100 59 180)
@@
 			)
 		)
-		(property "Footprint" "aliexpress:ESP32-C3-Super-Mini-Castellated-SMD-only"
+		(property "Footprint" "modules:ESP32-C3-Super-Mini-Castellated-SMD-only"
 			(at 0 0 0)
 			(unlocked yes)
@@
 			)
 		)
-		(model "${KIPRJMOD}/libraries/aliexpress.3dshapes/ESP32-C3-SuperMini.step"
+		(model "${KIPRJMOD}/libraries/modules.3dshapes/ESP32-C3-SuperMini.step"
 			(offset
 				(xyz 0 -2.3 0)

Commit message: Migrate JST SH connector footprints from `custom` to `connectors` library
Parts:
- J5: footprint custom:JST_SH_SM08B-SRSS-TB_1x08-1MP_P1.00mm_Horizontal -> connectors:JST_SH_SM08B-SRSS-TB_1x08-1MP_P1.00mm_Horizontal
Changed lines of the file:
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@@
 		)
 	)
-	(footprint "custom:JST_SH_SM08B-SRSS-TB_1x08-1MP_P1.00mm_Horizontal"
+	(footprint "connectors:JST_SH_SM08B-SRSS-TB_1x08-1MP_P1.00mm_Horizontal"
 		(layer "F.Cu")
 		(at 100 59)
@@
 			)
 		)
-		(property "Footprint" "custom:JST_SH_SM08B-SRSS-TB_1x08-1MP_P1.00mm_Horizontal"
+		(property "Footprint" "connectors:JST_SH_SM08B-SRSS-TB_1x08-1MP_P1.00mm_Horizontal"
 			(at 0 0 0)
 			(unlocked yes)
