File: dev/stackable2/lcd-round/lcd-round.kicad_pcb (KiCad board)
At the start: 2 copper layers, 35 x 35 mm, 16 parts, among them J1 JST SH, J2 Pin headers, J3 Pin headers, Q1 BSS138

Commit message: Migrate GC9A01 symbol and FPC footprint to modules
Parts:
- LCD1: footprint aliexpress:GC9A01-screen-connector-pads -> modules:GC9A01-screen-connector-pads
Changed lines of the file:
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@@
 		)
 	)
-	(footprint "aliexpress:GC9A01-screen-connector-pads"
+	(footprint "modules:GC9A01-screen-connector-pads"
 		(layer "B.Cu")
 		(at 99.95 80.9 90)
@@
 			)
 		)
-		(property "Footprint" "aliexpress:GC9A01-screen-connector-pads"
+		(property "Footprint" "modules:GC9A01-screen-connector-pads"
 			(at 0 0 -90)
 			(layer "F.Fab")
@@
 			(pintype "passive")
 		)
-		(model "${KIPRJMOD}/libraries/aliexpress.3dshapes/GC9A01-screen-alt.step"
+		(model "${KIPRJMOD}/libraries/modules.3dshapes/GC9A01-screen-alt.step"
 			(hide yes)
 			(offset
@@
 			)
 		)
-		(model "${KIPRJMOD}/libraries/aliexpress.3dshapes/GC9A01-screen.step"
+		(model "${KIPRJMOD}/libraries/modules.3dshapes/GC9A01-screen.step"
 			(offset
 				(xyz 10.6 0.3 -1)

Commit message: Migrate JST SH connector footprints from `custom` to `connectors` library
Parts:
- J1: footprint custom:JST_SH_SM08B-SRSS-TB_1x08-1MP_P1.00mm_Horizontal -> connectors:JST_SH_SM08B-SRSS-TB_1x08-1MP_P1.00mm_Horizontal
Changed lines of the file:
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@@
 		)
 	)
-	(footprint "custom:JST_SH_SM08B-SRSS-TB_1x08-1MP_P1.00mm_Horizontal"
+	(footprint "connectors:JST_SH_SM08B-SRSS-TB_1x08-1MP_P1.00mm_Horizontal"
 		(layer "B.Cu")
 		(at 100 58 180)
@@
 			)
 		)
-		(property "Footprint" "custom:JST_SH_SM08B-SRSS-TB_1x08-1MP_P1.00mm_Horizontal"
+		(property "Footprint" "connectors:JST_SH_SM08B-SRSS-TB_1x08-1MP_P1.00mm_Horizontal"
 			(at 0 0 0)
 			(unlocked yes)
