File: dev/stackable2/lcd-round/lcd-round.kicad_sch (KiCad schematic)
At the start: 10 parts, among them J1 JST SH, J2 Pin headers, J3 Pin headers, Q1 BSS138

Commit message: Migrate GC9A01 symbol and FPC footprint to modules
Parts:
- LCD1: footprint aliexpress:GC9A01-screen-connector-pads -> modules:GC9A01-screen-connector-pads; symbol aliexpress:LCD-round-1.28in-GC9A01 -> modules:LCD-round-1.28in-GC9A01
Changed lines of the file:
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@@
 	)
 	(symbol
-		(lib_id "aliexpress:LCD-round-1.28in-GC9A01")
+		(lib_id "modules:LCD-round-1.28in-GC9A01")
 		(at 132.08 87.63 0)
 		(unit 1)
@@
 			)
 		)
-		(property "Footprint" "aliexpress:GC9A01-screen-connector-pads"
+		(property "Footprint" "modules:GC9A01-screen-connector-pads"
 			(at 132.588 93.726 0)
 			(effects

Commit message: Migrate JST SH connector footprints from `custom` to `connectors` library
Parts:
- J1: footprint custom:JST_SH_SM08B-SRSS-TB_1x08-1MP_P1.00mm_Horizontal -> connectors:JST_SH_SM08B-SRSS-TB_1x08-1MP_P1.00mm_Horizontal
Changed lines of the file:
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@@
 			)
 		)
-		(property "Footprint" "custom:JST_SH_SM08B-SRSS-TB_1x08-1MP_P1.00mm_Horizontal"
+		(property "Footprint" "connectors:JST_SH_SM08B-SRSS-TB_1x08-1MP_P1.00mm_Horizontal"
 			(at 193.04 105.41 0)
 			(effects
