File: dev/power/ip5306-ups/ip5306-ups.kicad_pcb (KiCad board)
At the start: 2 copper layers, 110 x 44 mm, 64 parts, among them J1 USB_C_Receptacle_PowerOnly_6P, J10 Conn_01x02, J11 Conn_01x01, J12 Conn_01x01, J2 USB_C_Receptacle_PowerOnly_6P, J3 Barrel_Jack_Switch, J4 Screw_Terminal_01x02, J5 Conn_01x01, J6 Barrel_Jack_Switch, J7 Screw_Terminal_01x02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

Commit message: Move JLCPCB PCBA tooling hole footprint from `custom` to `mechanical`
Parts:
- REF** (x4): value jlcpcb-pcba-tooling-hole -> JLCPCB-PCBA-Tooling-Hole; footprint custom:jlcpcb-pcba-tooling-hole -> mechanical:JLCPCB-PCBA-Tooling-Hole
Changed lines of the file:
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@@
 		)
 	)
-	(footprint "custom:jlcpcb-pcba-tooling-hole"
+	(footprint "mechanical:JLCPCB-PCBA-Tooling-Hole"
 		(layer "F.Cu")
 		(at 190 113.5)
@@
 			)
 		)
-		(property "Value" "jlcpcb-pcba-tooling-hole"
+		(property "Value" "JLCPCB-PCBA-Tooling-Hole"
 			(at 0 1 0)
 			(unlocked yes)
@@
 			)
 		)
-		(property "Footprint" "custom:jlcpcb-pcba-tooling-hole"
+		(property "Footprint" "mechanical:JLCPCB-PCBA-Tooling-Hole"
 			(at 0 0 0)
 			(unlocked yes)
@@
 		)
 	)
-	(footprint "custom:jlcpcb-pcba-tooling-hole"
+	(footprint "mechanical:JLCPCB-PCBA-Tooling-Hole"
 		(layer "F.Cu")
 		(at 195 81.5)
@@
 			)
 		)
-		(property "Value" "jlcpcb-pcba-tooling-hole"
+		(property "Value" "JLCPCB-PCBA-Tooling-Hole"
 			(at 0 1 0)
 			(unlocked yes)
@@
 			)
 		)
-		(property "Footprint" "custom:jlcpcb-pcba-tooling-hole"
+		(property "Footprint" "mechanical:JLCPCB-PCBA-Tooling-Hole"
 			(at 0 0 0)
 			(unlocked yes)
@@
 		)
 	)
-	(footprint "custom:jlcpcb-pcba-tooling-hole"
+	(footprint "mechanical:JLCPCB-PCBA-Tooling-Hole"
 		(layer "F.Cu")
 		(at 97 113.5)
@@
 			)
 		)
-		(property "Value" "jlcpcb-pcba-tooling-hole"
+		(property "Value" "JLCPCB-PCBA-Tooling-Hole"
 			(at 0 1 0)
 			(unlocked yes)
@@
 			)
 		)
-		(property "Footprint" "custom:jlcpcb-pcba-tooling-hole"
+		(property "Footprint" "mechanical:JLCPCB-PCBA-Tooling-Hole"
 			(at 0 0 0)
 			(unlocked yes)
@@
 		)
 	)
-	(footprint "custom:jlcpcb-pcba-tooling-hole"
+	(footprint "mechanical:JLCPCB-PCBA-Tooling-Hole"
 		(layer "F.Cu")
 		(at 92 81.5)
@@
 			)
 		)
-		(property "Value" "jlcpcb-pcba-tooling-hole"
+		(property "Value" "JLCPCB-PCBA-Tooling-Hole"
 			(at 0 1 0)
 			(unlocked yes)
@@
 			)
 		)
-		(property "Footprint" "custom:jlcpcb-pcba-tooling-hole"
+		(property "Footprint" "mechanical:JLCPCB-PCBA-Tooling-Hole"
 			(at 0 0 0)
 			(unlocked yes)
