File: pcb-archived/power/ip5306-ups/ip5306-ups.kicad_pcb (KiCad board)
At the start: 2 copper layers, 110 x 44 mm, 64 parts, among them J1 USB_C_Receptacle_PowerOnly_6P, J10 Conn_01x02, J11 Conn_01x01, J12 Conn_01x01, J2 USB_C_Receptacle_PowerOnly_6P, J3 Barrel_Jack_Switch, J4 Screw_Terminal_01x02, J5 Conn_01x01, J6 Barrel_Jack_Switch, J7 Screw_Terminal_01x02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

Commit message: Fix DRC warnings
Changed lines of the file:
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@@
 		(layer "F.Cu")
 		(at 163.4435 78.166 180)
-		(descr "SOT, 6 Pin (https://www.jedec.org/sites/default/files/docs/Mo-178c.PDF variant AB), generated with kicad-footprint-generator ipc_gullwing_generator.py")
+		(descr "SOT, 6 Pin (~), generated with kicad-footprint-generator ipc_gullwing_generator.py")
 		(tags "SOT TO_SOT_SMD")
 		(property "Reference" "U3"
-			(at 0 -2.4 360)
+			(at 0 -2.4 0)
 			(layer "F.SilkS")
 			(hide yes)
@@
 		)
 		(property "Value" "MT3608"
-			(at 0 2.4 360)
+			(at 0 2.4 0)
 			(layer "F.Fab")
 			(effects
@@
 		)
 		(fp_text user "${REFERENCE}"
-			(at 0 0 360)
+			(at 0 0 0)
 			(layer "F.Fab")
 			(effects
@@
 			(layer "F.SilkS")
 		)
+		(fp_poly
+			(pts
+				(xy -3.5 -3.3) (xy 3.5 -3.3) (xy 3.5 -1.7) (xy 4.3 -1.7) (xy 4.3 1.7) (xy 3.5 1.7) (xy 3.5 3.3)
+				(xy -3.5 3.3) (xy -3.5 1.7) (xy -4.3 1.7) (xy -4.3 -1.7) (xy -3.5 -1.7)
+			)
+			(stroke
+				(width 0.05)
+				(type solid)
+			)
+			(fill none)
+			(layer "F.CrtYd")
+		)
 		(fp_circle
 			(center -3.5 3.3)
@@
 			(size 3.775 3.2)
 			(layers "F.Cu" "F.Paste" "F.Mask")
-			(roundrect_rratio 0.078125)
+			(roundrect_rratio 0.125)
 			(net 9 "SW")
 			(pinfunction "1")
@@
 			(size 3.775 3.225)
 			(layers "F.Cu" "F.Paste" "F.Mask")
-			(roundrect_rratio 0.07751937984)
+			(roundrect_rratio 0.125)
 			(net 2 "B+")
 			(pinfunction "2")
@@
 		(tags "SOT TO_SOT_SMD")
 		(property "Reference" "Q2"
-			(at 0 -2.4 360)
+			(at 0 -2.4 0)
 			(layer "F.SilkS")
 			(hide yes)
@@
 		)
 		(property "Value" "AO3401A"
-			(at 0 2.4 360)
+			(at 0 2.4 0)
 			(layer "F.Fab")
 			(effects
@@
 		)
 		(fp_text user "${REFERENCE}"
-			(at 0 0 360)
+			(at 0 0 0)
 			(layer "F.Fab")
 			(effects
@@
 		(at 143.51 99.04)
 		(property "Reference" "BT1"
-			(at 0 -4 360)
+			(at 0 -4 0)
 			(layer "F.SilkS")
 			(hide yes)
@@
 		)
 		(property "Value" "Battery_Cell"
-			(at 0 4 360)
+			(at 0 4 0)
 			(layer "F.Fab")
 			(effects
@@
 		)
 		(property "Footprint" "lcsc:BAT-TH_18650-A5BJ001"
-			(at 0 0 360)
+			(at 0 0 0)
 			(layer "F.Fab")
 			(hide yes)
@@
 		)
 		(property "Datasheet" ""
-			(at 0 0 360)
+			(at 0 0 0)
 			(layer "F.Fab")
 			(hide yes)
@@
 		)
 		(property "Description" "Single-cell battery"
-			(at 0 0 360)
+			(at 0 0 0)
 			(layer "F.Fab")
 			(hide yes)
@@
 		)
 		(fp_text user "${REFERENCE}"
-			(at 0 0 360)
+			(at 0 0 0)
 			(layer "F.Fab")
 			(effects
@@
 		(tags "SOT TO_SOT_SMD")
 		(property "Reference" "Q1"
-			(at 0 -2.4 360)
+			(at 0 -2.4 0)
 			(layer "F.SilkS")
 			(hide yes)
@@
 		)
 		(property "Value" "AO3401A"
-			(at 0 2.4 360)
+			(at 0 2.4 0)
 			(layer "F.Fab")
 			(effects
@@
 		)
 		(fp_text user "${REFERENCE}"
-			(at 0 0 360)
+			(at 0 0 0)
 			(layer "F.Fab")
 			(effects
@@
 		(tags "Diode SMA (DO-214AC)")
 		(property "Reference" "D1"
-			(at 0 -2.5 360)
+			(at 0 -2.5 0)
 			(layer "F.SilkS")
 			(hide yes)
@@
 		)
 		(property "Value" "SS34"
-			(at 0 2.6 360)
+			(at 0 2.6 0)
 			(layer "F.Fab")
 			(effects
@@
 		)
 		(fp_text user "${REFERENCE}"
-			(at 0 -2.5 360)
+			(at 0 -2.5 0)
 			(layer "F.Fab")
 			(effects
@@
 		(tags "resistor handsolder")
 		(property "Reference" "R2"
-			(at 0 -1.65 360)
+			(at 0 -1.65 0)
 			(layer "F.SilkS")
 			(hide yes)
@@
 		)
 		(property "Value" "20R"
-			(at 0 1.65 360)
+			(at 0 1.65 0)
 			(layer "F.Fab")
 			(effects
@@
 		)
 		(fp_text user "${REFERENCE}"
-			(at 0 0 360)
+			(at 0 0 0)
 			(layer "F.Fab")
 			(effects
@@
 		(at 141.01 81.28 180)
 		(property "Reference" "J10"
-			(at 0 -4 360)
+			(at 0 -4 0)
 			(layer "F.SilkS")
 			(hide yes)
@@
 		)
 		(property "Value" "Conn_01x02"
-			(at 0 4 360)
+			(at 0 4 0)
 			(layer "F.Fab")
 			(effects
@@
 		)
 		(property "Footprint" "custom:JST_XH_S2B-XH-2AW_1x02_P2.50mm_pad2gnd"
-			(at 0 0 360)
+			(at 0 0 0)
 			(layer "F.Fab")
 			(hide yes)
@@
 		)
 		(property "Datasheet" ""
-			(at 0 0 360)
+			(at 0 0 0)
 			(layer "F.Fab")
 			(hide yes)
@@
 		)
 		(property "Description" "Generic connector, single row, 01x02, script generated (kicad-library-utils/schlib/autogen/connector/)"
-			(at 0 0 360)
+			(at 0 0 0)
 			(layer "F.Fab")
 			(hide yes)
@@
 		)
 		(fp_text user "${REFERENCE}"
-			(at 0 0 360)
+			(at 0 0 0)
 			(layer "F.Fab")
 			(effects
@@
 		(at 161.846 83.566)
 		(property "Reference" "L2"
-			(at 0 -4 360)
+			(at 0 -4 0)
 			(layer "F.SilkS")
 			(hide yes)
@@
 		)
 		(property "Value" "22uH"
-			(at 0 4 360)
+			(at 0 4 0)
 			(layer "F.Fab")
 			(effects
@@
 		)
 		(property "Footprint" "lcsc:IND-SMD_L7.0-W6.6"
-			(at 0 0 360)
+			(at 0 0 0)
 			(layer "F.Fab")
 			(hide yes)
@@
 		)
 		(property "Datasheet" ""
-			(at 0 0 360)
+			(at 0 0 0)
 			(layer "F.Fab")
 			(hide yes)
@@
 		)
 		(property "Description" "Inductor"
-			(at 0 0 360)
+			(at 0 0 0)
 			(layer "F.Fab")
 			(hide yes)
@@
 			(layer "F.SilkS")
 		)
+		(fp_poly
+			(pts
+				(xy -3.5 -3.3) (xy -3.5 -1.7) (xy -4.3 -1.7) (xy -4.3 1.7) (xy -3.5 1.7) (xy -3.49 3.3) (xy 3.5 3.3)
+				(xy 3.5 1.7) (xy 4.3 1.7) (xy 4.3 -1.7) (xy 3.5 -1.7) (xy 3.5 -3.3)
+			)
+			(stroke
+				(width 0.05)
+				(type solid)
+			)
+			(fill none)
+			(layer "F.CrtYd")
+		)
 		(fp_circle
 			(center -3.5 3.3)
@@
 		)
 		(fp_text user "${REFERENCE}"
-			(at 0 0 360)
+			(at 0 0 0)
 			(layer "F.Fab")
 			(effects
@@
 			)
 		)
-		(pad "1" smd rect
+		(pad "1" smd roundrect
 			(at -3 0)
 			(size 2.4 3.2)
 			(layers "F.Cu" "F.Paste" "F.Mask")
+			(roundrect_rratio 0.125)
 			(net 5 "BOOST")
 			(pinfunction "1")
 			(pintype "passive")
 		)
-		(pad "2" smd rect
+		(pad "2" smd roundrect
 			(at 3 0)
 			(size 2.4 3.2)
 			(layers "F.Cu" "F.Paste" "F.Mask")
+			(roundrect_rratio 0.125)
 			(net 34 "BOOST_SW")
 			(pinfunction "2")
@@
 		(tags "SOT TO_SOT_SMD")
 		(property "Reference" "Q3"
-			(at 0 -2.4 360)
+			(at 0 -2.4 0)
 			(layer "F.SilkS")
 			(hide yes)
@@
 		)
 		(property "Value" "AO3400A"
-			(at 0 2.4 360)
+			(at 0 2.4 0)
 			(layer "F.Fab")
 			(effects
@@
 		)
 		(fp_text user "${REFERENCE}"
-			(at 0 0 360)
+			(at 0 0 0)
 			(layer "F.Fab")
 			(effects
@@
 		(tags "THT Terminal Block Phoenix MKDS-1,5-2-5.08 pitch 5.08mm size 10.2x9.8mm^2 drill 1.3mm pad 2.6mm")
 		(property "Reference" "J4"
-			(at 2.54 -6.26 360)
+			(at 2.54 -6.26 0)
 			(layer "F.SilkS")
 			(hide yes)
@@
 		)
 		(property "Value" "Screw_Terminal_01x02"
-			(at 2.54 5.66 360)
+			(at 2.54 5.66 0)
 			(layer "F.Fab")
 			(effects
@@
 		)
 		(fp_text user "${REFERENCE}"
-			(at 2.54 3.2 360)
+			(at 2.54 3.2 0)
 			(layer "F.Fab")
 			(effects
@@
 		(tags "SOT TO_SOT_SMD")
 		(property "Reference" "U2"
-			(at 0 -2.4 360)
+			(at 0 -2.4 0)
 			(layer "F.SilkS")
 			(hide yes)
@@
 		)
 		(property "Value" "XB5350D0"
-			(at 0 2.4 360)
+			(at 0 2.4 0)
 			(layer "F.Fab")
 			(effects
@@
 		)
 		(fp_text user "${REFERENCE}"
-			(at 0 0 360)
+			(at 0 0 0)
 			(layer "F.Fab")
 			(effects
@@
 		(at 131.2895 113.1395)
 		(property "Reference" "LED5"
-			(at 0 -4 360)
+			(at 0 -4 0)
 			(layer "F.SilkS")
 			(hide yes)
@@
 		)
 		(property "Value" "~"
-			(at 0 4 360)
+			(at 0 4 0)
 			(layer "F.Fab")
 			(effects
@@
 		)
 		(property "Footprint" "lcsc:LED-SMD_3P-L5.7-W3.0-RD"
-			(at 0 0 360)
+			(at 0 0 0)
 			(layer "F.Fab")
 			(hide yes)
@@
 		)
 		(property "Datasheet" ""
-			(at 0 0 360)
+			(at 0 0 0)
 			(layer "F.Fab")
 			(hide yes)
@@
 		)
 		(property "Description" "Light emitting diode"
-			(at 0 0 360)
+			(at 0 0 0)
 			(layer "F.Fab")
 			(hide yes)
@@
 			(layer "F.SilkS")
 		)
+		(fp_rect
+			(start -3.6 -1.6)
+			(end 3.6 1.6)
+			(stroke
+				(width 0.05)
+				(type default)
+			)
+			(fill none)
+			(layer "F.CrtYd")
+		)
 		(fp_circle
 			(center -2.85 1.5)
@@
 		)
 		(fp_text user "${REFERENCE}"
-			(at 0 0 360)
+			(at 0 0 0)
 			(layer "F.Fab")
 			(effects
@@
 		(tags "THT Terminal Block Phoenix MKDS-1,5-2-5.08 pitch 5.08mm size 10.2x9.8mm^2 drill 1.3mm pad 2.6mm")
 		(property "Reference" "J7"
-			(at 2.54 -6.26 360)
+			(at 2.54 -6.26 0)
 			(layer "F.SilkS")
 			(hide yes)
@@
 		)
 		(property "Value" "Screw_Terminal_01x02"
-			(at 2.54 5.66 360)
+			(at 2.54 5.66 0)
 			(layer "F.Fab")
 			(effects
@@
 		)
 		(fp_text user "${REFERENCE}"
-			(at 2.54 3.2 360)
+			(at 2.54 3.2 0)
 			(layer "F.Fab")
 			(effects
