File: pcb/jigs/reflow/reflow.kicad_sch (KiCad schematic)
At the start: 62 parts, among them J1 Pin headers, J2 Pin headers, Q1 SDV301N3, Q2 SDV301N3, Q3 SDV301N3, Q4 SDV301N3, Q5 SDV301N3, Q6 SDV301N3, Q7 SDV301N3, Q8 SDV301N3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

Commit message: Migrate `C_0402_1005Metric` footprint to `passives`
Parts:
- C0, C1, C2: footprint custom:C_0402_1005Metric_simple -> passives:C_0402_1005Metric
Changed lines of the file:
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@@
 			)
 		)
-		(property "Footprint" "custom:C_0402_1005Metric_simple"
+		(property "Footprint" "passives:C_0402_1005Metric"
 			(at 57.15 77.47 0)
 			(effects
@@
 			)
 		)
-		(property "Footprint" "custom:C_0402_1005Metric_simple"
+		(property "Footprint" "passives:C_0402_1005Metric"
 			(at 214.63 35.56 0)
 			(effects
@@
 			)
 		)
-		(property "Footprint" "custom:C_0402_1005Metric_simple"
+		(property "Footprint" "passives:C_0402_1005Metric"
 			(at 35.56 77.47 0)
 			(effects

Commit message: Migrate `LED_0402_1005Metric` footprint to `passives`
Parts:
- D1, D10, D11, D12, D13, D2, D3, D4, D5, D6, D7, D8, D9: footprint custom:LED_0402_1005Metric -> passives:LED_0402_1005Metric
Changed lines of the file:
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@@
 			)
 		)
-		(property "Footprint" "custom:LED_0402_1005Metric"
+		(property "Footprint" "passives:LED_0402_1005Metric"
 			(at 25.4 161.29 90)
 			(effects
@@
 			)
 		)
-		(property "Footprint" "custom:LED_0402_1005Metric"
+		(property "Footprint" "passives:LED_0402_1005Metric"
 			(at 25.4 106.68 90)
 			(effects
@@
 			)
 		)
-		(property "Footprint" "custom:LED_0402_1005Metric"
+		(property "Footprint" "passives:LED_0402_1005Metric"
 			(at 78.74 161.29 90)
 			(effects
@@
 			)
 		)
-		(property "Footprint" "custom:LED_0402_1005Metric"
+		(property "Footprint" "passives:LED_0402_1005Metric"
 			(at 13.97 106.68 90)
 			(effects
@@
 			)
 		)
-		(property "Footprint" "custom:LED_0402_1005Metric"
+		(property "Footprint" "passives:LED_0402_1005Metric"
 			(at 90.17 106.68 90)
 			(effects
@@
 			)
 		)
-		(property "Footprint" "custom:LED_0402_1005Metric"
+		(property "Footprint" "passives:LED_0402_1005Metric"
 			(at 62.23 168.91 90)
 			(effects
@@
 			)
 		)
-		(property "Footprint" "custom:LED_0402_1005Metric"
+		(property "Footprint" "passives:LED_0402_1005Metric"
 			(at 127 168.91 90)
 			(effects
@@
 			)
 		)
-		(property "Footprint" "custom:LED_0402_1005Metric"
+		(property "Footprint" "passives:LED_0402_1005Metric"
 			(at 62.23 114.3 90)
 			(effects
@@
 			)
 		)
-		(property "Footprint" "custom:LED_0402_1005Metric"
+		(property "Footprint" "passives:LED_0402_1005Metric"
 			(at 90.17 161.29 90)
 			(effects
@@
 			)
 		)
-		(property "Footprint" "custom:LED_0402_1005Metric"
+		(property "Footprint" "passives:LED_0402_1005Metric"
 			(at 78.74 106.68 90)
 			(effects
@@
 			)
 		)
-		(property "Footprint" "custom:LED_0402_1005Metric"
+		(property "Footprint" "passives:LED_0402_1005Metric"
 			(at 13.97 161.29 90)
 			(effects
@@
 			)
 		)
-		(property "Footprint" "custom:LED_0402_1005Metric"
+		(property "Footprint" "passives:LED_0402_1005Metric"
 			(at 259.08 49.53 90)
 			(effects
@@
 			)
 		)
-		(property "Footprint" "custom:LED_0402_1005Metric"
+		(property "Footprint" "passives:LED_0402_1005Metric"
 			(at 127 114.3 90)
 			(effects

Commit message: Migrate `DFN1006-3` footprint to `packages`
Parts:
- Q1, Q2, Q3, Q4, Q5, Q6, Q7, Q8, Q9: footprint custom:DFN1006-3 -> packages:DFN1006-3
Changed lines of the file:
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@@
 			)
 		)
-		(property "Footprint" "custom:DFN1006-3"
+		(property "Footprint" "packages:DFN1006-3"
 			(at 142.875 45.72 0)
 			(effects
@@
 			)
 		)
-		(property "Footprint" "custom:DFN1006-3"
+		(property "Footprint" "packages:DFN1006-3"
 			(at 171.45 156.845 0)
 			(effects
@@
 			)
 		)
-		(property "Footprint" "custom:DFN1006-3"
+		(property "Footprint" "packages:DFN1006-3"
 			(at 273.05 102.235 0)
 			(effects
@@
 			)
 		)
-		(property "Footprint" "custom:DFN1006-3"
+		(property "Footprint" "packages:DFN1006-3"
 			(at 273.05 156.845 0)
 			(effects
@@
 			)
 		)
-		(property "Footprint" "custom:DFN1006-3"
+		(property "Footprint" "packages:DFN1006-3"
 			(at 149.86 156.845 0)
 			(effects
@@
 			)
 		)
-		(property "Footprint" "custom:DFN1006-3"
+		(property "Footprint" "packages:DFN1006-3"
 			(at 171.45 102.235 0)
 			(effects
@@
 			)
 		)
-		(property "Footprint" "custom:DFN1006-3"
+		(property "Footprint" "packages:DFN1006-3"
 			(at 149.86 102.235 0)
 			(effects
@@
 			)
 		)
-		(property "Footprint" "custom:DFN1006-3"
+		(property "Footprint" "packages:DFN1006-3"
 			(at 251.46 156.845 0)
 			(effects
@@
 			)
 		)
-		(property "Footprint" "custom:DFN1006-3"
+		(property "Footprint" "packages:DFN1006-3"
 			(at 251.46 102.235 0)
 			(effects

Commit message: Migrate `FSOP-8_L3.3-W1.7-P0.80-LS2.9-BL` footprint to `packages`
Parts:
- U1: footprint lcsc:FSOP-8_L3.3-W1.7-P0.80-LS2.9-BL -> packages:FSOP-8_L3.3-W1.7-P0.80-LS2.9-BL
Changed lines of the file:
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@@
 			)
 		)
-		(property "Footprint" "lcsc:FSOP-8_L3.3-W1.7-P0.80-LS2.9-BL"
+		(property "Footprint" "packages:FSOP-8_L3.3-W1.7-P0.80-LS2.9-BL"
 			(at 203.2 52.07 0)
 			(effects

Commit message: Migrate `X2-DFN1010-6_L1.0-W1.0-P0.35-BL` footprint to `packages`
Parts:
- U4: footprint lcsc:X2-DFN1010-6_L1.0-W1.0-P0.35-BL -> packages:X2-DFN1010-6_L1.0-W1.0-P0.35-BL
Changed lines of the file:
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@@
 			)
 		)
-		(property "Footprint" "lcsc:X2-DFN1010-6_L1.0-W1.0-P0.35-BL"
+		(property "Footprint" "packages:X2-DFN1010-6_L1.0-W1.0-P0.35-BL"
 			(at 212.09 85.09 0)
 			(effects
@@
 			)
 		)
-		(property "Footprint" "lcsc:X2-DFN1010-6_L1.0-W1.0-P0.35-BL"
+		(property "Footprint" "packages:X2-DFN1010-6_L1.0-W1.0-P0.35-BL"
 			(at 212.09 139.7 0)
 			(effects
@@
 			)
 		)
-		(property "Footprint" "lcsc:X2-DFN1010-6_L1.0-W1.0-P0.35-BL"
+		(property "Footprint" "packages:X2-DFN1010-6_L1.0-W1.0-P0.35-BL"
 			(at 210.82 109.22 0)
 			(effects

Commit message: Migrate `X2-DFN1210-8_L1.2-W1.0-P0.30-BL` footprint to `packages`
Parts:
- U3: footprint lcsc:X2-DFN1210-8_L1.2-W1.0-P0.30-BL -> packages:X2-DFN1210-8_L1.2-W1.0-P0.30-BL
Changed lines of the file:
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@@
 			)
 		)
-		(property "Footprint" "lcsc:X2-DFN1210-8_L1.2-W1.0-P0.30-BL"
+		(property "Footprint" "packages:X2-DFN1210-8_L1.2-W1.0-P0.30-BL"
 			(at 111.76 125.73 0)
 			(effects
@@
 			)
 		)
-		(property "Footprint" "lcsc:X2-DFN1210-8_L1.2-W1.0-P0.30-BL"
+		(property "Footprint" "packages:X2-DFN1210-8_L1.2-W1.0-P0.30-BL"
 			(at 114.3 156.21 0)
 			(effects
@@
 			)
 		)
-		(property "Footprint" "lcsc:X2-DFN1210-8_L1.2-W1.0-P0.30-BL"
+		(property "Footprint" "packages:X2-DFN1210-8_L1.2-W1.0-P0.30-BL"
 			(at 114.3 101.6 0)
 			(effects

Commit message: Migrate `X2-DFN2010-8_L2.0-W1.0-P0.50-BL` footprint to `packages`
Parts:
- U2: footprint lcsc:X2-DFN2010-8_L2.0-W1.0-P0.50-BL -> packages:X2-DFN2010-8_L2.0-W1.0-P0.50-BL
Changed lines of the file:
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@@
 			)
 		)
-		(property "Footprint" "lcsc:X2-DFN2010-8_L2.0-W1.0-P0.50-BL"
+		(property "Footprint" "packages:X2-DFN2010-8_L2.0-W1.0-P0.50-BL"
 			(at 49.53 101.6 0)
 			(effects
@@
 			)
 		)
-		(property "Footprint" "lcsc:X2-DFN2010-8_L2.0-W1.0-P0.50-BL"
+		(property "Footprint" "packages:X2-DFN2010-8_L2.0-W1.0-P0.50-BL"
 			(at 48.26 125.73 0)
 			(effects
@@
 			)
 		)
-		(property "Footprint" "lcsc:X2-DFN2010-8_L2.0-W1.0-P0.50-BL"
+		(property "Footprint" "packages:X2-DFN2010-8_L2.0-W1.0-P0.50-BL"
 			(at 49.53 156.21 0)
 			(effects

Commit message: Migrate `LED_0402_1005Metric` footprint to `led`
Parts:
- D1, D10, D11, D12, D13, D2, D3, D4, D5, D6, D7, D8, D9: footprint passives:LED_0402_1005Metric -> led:LED_0402_1005Metric
Changed lines of the file:
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@@
 			)
 		)
-		(property "Footprint" "passives:LED_0402_1005Metric"
+		(property "Footprint" "led:LED_0402_1005Metric"
 			(at 25.4 161.29 90)
 			(effects
@@
 			)
 		)
-		(property "Footprint" "passives:LED_0402_1005Metric"
+		(property "Footprint" "led:LED_0402_1005Metric"
 			(at 25.4 106.68 90)
 			(effects
@@
 			)
 		)
-		(property "Footprint" "passives:LED_0402_1005Metric"
+		(property "Footprint" "led:LED_0402_1005Metric"
 			(at 78.74 161.29 90)
 			(effects
@@
 			)
 		)
-		(property "Footprint" "passives:LED_0402_1005Metric"
+		(property "Footprint" "led:LED_0402_1005Metric"
 			(at 13.97 106.68 90)
 			(effects
@@
 			)
 		)
-		(property "Footprint" "passives:LED_0402_1005Metric"
+		(property "Footprint" "led:LED_0402_1005Metric"
 			(at 90.17 106.68 90)
 			(effects
@@
 			)
 		)
-		(property "Footprint" "passives:LED_0402_1005Metric"
+		(property "Footprint" "led:LED_0402_1005Metric"
 			(at 62.23 168.91 90)
 			(effects
@@
 			)
 		)
-		(property "Footprint" "passives:LED_0402_1005Metric"
+		(property "Footprint" "led:LED_0402_1005Metric"
 			(at 127 168.91 90)
 			(effects
@@
 			)
 		)
-		(property "Footprint" "passives:LED_0402_1005Metric"
+		(property "Footprint" "led:LED_0402_1005Metric"
 			(at 62.23 114.3 90)
 			(effects
@@
 			)
 		)
-		(property "Footprint" "passives:LED_0402_1005Metric"
+		(property "Footprint" "led:LED_0402_1005Metric"
 			(at 90.17 161.29 90)
 			(effects
@@
 			)
 		)
-		(property "Footprint" "passives:LED_0402_1005Metric"
+		(property "Footprint" "led:LED_0402_1005Metric"
 			(at 78.74 106.68 90)
 			(effects
@@
 			)
 		)
-		(property "Footprint" "passives:LED_0402_1005Metric"
+		(property "Footprint" "led:LED_0402_1005Metric"
 			(at 13.97 161.29 90)
 			(effects
@@
 			)
 		)
-		(property "Footprint" "passives:LED_0402_1005Metric"
+		(property "Footprint" "led:LED_0402_1005Metric"
 			(at 259.08 49.53 90)
 			(effects
@@
 			)
 		)
-		(property "Footprint" "passives:LED_0402_1005Metric"
+		(property "Footprint" "led:LED_0402_1005Metric"
 			(at 127 114.3 90)
 			(effects
