File: pcb/jigs/logic-led-jig/logic-led-jig.kicad_pcb (KiCad board)
At the start: 2 copper layers, 19.1 x 22.9 mm, 22 parts, among them J1 Conn_01x08, J2 Conn_01x02, Q1 AO3404, Q2 AO3404, Q3 AO3404, Q4 AO3404, Q5 AO3404, Q6 AO3404, Q7 AO3404, Q8 AO3404

Commit message: Migrate `LED_0805_2012Metric` footprint to `passives`
Parts:
- D1, D2, D3, D4, D5, D6, D7, D8: footprint custom:LED_0805_2012Metric_simple -> passives:LED_0805_2012Metric
Changed lines of the file:
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@@
 		)
 	)
-	(footprint "custom:LED_0805_2012Metric_simple"
+	(footprint "passives:LED_0805_2012Metric"
 		(layer "F.Cu")
 		(at 138.898 91.44 180)
@@
 			)
 		)
-		(property "Footprint" "custom:LED_0805_2012Metric_simple"
+		(property "Footprint" "passives:LED_0805_2012Metric"
 			(at 0 0 180)
 			(unlocked yes)
@@
 		)
 	)
-	(footprint "custom:LED_0805_2012Metric_simple"
+	(footprint "passives:LED_0805_2012Metric"
 		(layer "F.Cu")
 		(at 138.938 83.82 180)
@@
 			)
 		)
-		(property "Footprint" "custom:LED_0805_2012Metric_simple"
+		(property "Footprint" "passives:LED_0805_2012Metric"
 			(at 0 0 180)
 			(unlocked yes)
@@
 		)
 	)
-	(footprint "custom:LED_0805_2012Metric_simple"
+	(footprint "passives:LED_0805_2012Metric"
 		(layer "F.Cu")
 		(at 138.898 96.52 180)
@@
 			)
 		)
-		(property "Footprint" "custom:LED_0805_2012Metric_simple"
+		(property "Footprint" "passives:LED_0805_2012Metric"
 			(at 0 0 180)
 			(unlocked yes)
@@
 		)
 	)
-	(footprint "custom:LED_0805_2012Metric_simple"
+	(footprint "passives:LED_0805_2012Metric"
 		(layer "F.Cu")
 		(at 138.938 81.28 180)
@@
 			)
 		)
-		(property "Footprint" "custom:LED_0805_2012Metric_simple"
+		(property "Footprint" "passives:LED_0805_2012Metric"
 			(at 0 0 180)
 			(unlocked yes)
@@
 		)
 	)
-	(footprint "custom:LED_0805_2012Metric_simple"
+	(footprint "passives:LED_0805_2012Metric"
 		(layer "F.Cu")
 		(at 138.898 88.9 180)
@@
 			)
 		)
-		(property "Footprint" "custom:LED_0805_2012Metric_simple"
+		(property "Footprint" "passives:LED_0805_2012Metric"
 			(at 0 0 180)
 			(unlocked yes)
@@
 		)
 	)
-	(footprint "custom:LED_0805_2012Metric_simple"
+	(footprint "passives:LED_0805_2012Metric"
 		(layer "F.Cu")
 		(at 138.898 93.98 180)
@@
 			)
 		)
-		(property "Footprint" "custom:LED_0805_2012Metric_simple"
+		(property "Footprint" "passives:LED_0805_2012Metric"
 			(at 0 0 180)
 			(unlocked yes)
@@
 		)
 	)
-	(footprint "custom:LED_0805_2012Metric_simple"
+	(footprint "passives:LED_0805_2012Metric"
 		(layer "F.Cu")
 		(at 138.938 86.36 180)
@@
 			)
 		)
-		(property "Footprint" "custom:LED_0805_2012Metric_simple"
+		(property "Footprint" "passives:LED_0805_2012Metric"
 			(at 0 0 180)
 			(unlocked yes)
@@
 		)
 	)
-	(footprint "custom:LED_0805_2012Metric_simple"
+	(footprint "passives:LED_0805_2012Metric"
 		(layer "F.Cu")
 		(at 138.938 78.74 180)
@@
 			)
 		)
-		(property "Footprint" "custom:LED_0805_2012Metric_simple"
+		(property "Footprint" "passives:LED_0805_2012Metric"
 			(at 0 0 180)
 			(unlocked yes)

Commit message: Migrate `LED_0805_2012Metric` footprint to `led`
Parts:
- D1, D2, D3, D4, D5, D6, D7, D8: footprint passives:LED_0805_2012Metric -> led:LED_0805_2012Metric
Changed lines of the file:
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@@
 		)
 	)
-	(footprint "passives:LED_0805_2012Metric"
+	(footprint "led:LED_0805_2012Metric"
 		(layer "F.Cu")
 		(at 138.898 91.44 180)
@@
 			)
 		)
-		(property "Footprint" "passives:LED_0805_2012Metric"
+		(property "Footprint" "led:LED_0805_2012Metric"
 			(at 0 0 180)
 			(unlocked yes)
@@
 		)
 	)
-	(footprint "passives:LED_0805_2012Metric"
+	(footprint "led:LED_0805_2012Metric"
 		(layer "F.Cu")
 		(at 138.938 83.82 180)
@@
 			)
 		)
-		(property "Footprint" "passives:LED_0805_2012Metric"
+		(property "Footprint" "led:LED_0805_2012Metric"
 			(at 0 0 180)
 			(unlocked yes)
@@
 		)
 	)
-	(footprint "passives:LED_0805_2012Metric"
+	(footprint "led:LED_0805_2012Metric"
 		(layer "F.Cu")
 		(at 138.898 96.52 180)
@@
 			)
 		)
-		(property "Footprint" "passives:LED_0805_2012Metric"
+		(property "Footprint" "led:LED_0805_2012Metric"
 			(at 0 0 180)
 			(unlocked yes)
@@
 		)
 	)
-	(footprint "passives:LED_0805_2012Metric"
+	(footprint "led:LED_0805_2012Metric"
 		(layer "F.Cu")
 		(at 138.938 81.28 180)
@@
 			)
 		)
-		(property "Footprint" "passives:LED_0805_2012Metric"
+		(property "Footprint" "led:LED_0805_2012Metric"
 			(at 0 0 180)
 			(unlocked yes)
@@
 		)
 	)
-	(footprint "passives:LED_0805_2012Metric"
+	(footprint "led:LED_0805_2012Metric"
 		(layer "F.Cu")
 		(at 138.898 88.9 180)
@@
 			)
 		)
-		(property "Footprint" "passives:LED_0805_2012Metric"
+		(property "Footprint" "led:LED_0805_2012Metric"
 			(at 0 0 180)
 			(unlocked yes)
@@
 		)
 	)
-	(footprint "passives:LED_0805_2012Metric"
+	(footprint "led:LED_0805_2012Metric"
 		(layer "F.Cu")
 		(at 138.898 93.98 180)
@@
 			)
 		)
-		(property "Footprint" "passives:LED_0805_2012Metric"
+		(property "Footprint" "led:LED_0805_2012Metric"
 			(at 0 0 180)
 			(unlocked yes)
@@
 		)
 	)
-	(footprint "passives:LED_0805_2012Metric"
+	(footprint "led:LED_0805_2012Metric"
 		(layer "F.Cu")
 		(at 138.938 86.36 180)
@@
 			)
 		)
-		(property "Footprint" "passives:LED_0805_2012Metric"
+		(property "Footprint" "led:LED_0805_2012Metric"
 			(at 0 0 180)
 			(unlocked yes)
@@
 		)
 	)
-	(footprint "passives:LED_0805_2012Metric"
+	(footprint "led:LED_0805_2012Metric"
 		(layer "F.Cu")
 		(at 138.938 78.74 180)
@@
 			)
 		)
-		(property "Footprint" "passives:LED_0805_2012Metric"
+		(property "Footprint" "led:LED_0805_2012Metric"
 			(at 0 0 180)
 			(unlocked yes)
