File: pcb-archived/stackable1/power-eta6003-5v-ups/power-eta6003-5v-ups.kicad_sch (KiCad schematic)
At the start: 54 parts, among them Q1 2N7002DW, Q2 AO3401A, SW1 SW_SPDT, U1 ETA6003, U2 XB3306D, U3 ME6211C33M5, U4 INA3221, U5 MT3608

Commit message: Rename `connectors` symbol and footprint libraries to `connector`
Parts:
- TH1: footprint connectors:JST_SH_SM02B-SRSS-TB_1x02-1MP_P1.00mm_Horizontal -> connector:JST_SH_SM02B-SRSS-TB_1x02-1MP_P1.00mm_Horizontal
Changed lines of the file:
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@@
 			)
 		)
-		(property "Footprint" "connectors:JST_SH_SM02B-SRSS-TB_1x02-1MP_P1.00mm_Horizontal"
+		(property "Footprint" "connector:JST_SH_SM02B-SRSS-TB_1x02-1MP_P1.00mm_Horizontal"
 			(at 45.72 34.29 0)
 			(effects
