File: pcb-archived/stackable1/relay-module-5v-half/relay-module-5v-half.kicad_sch (KiCad schematic)
At the start: 14 parts, among them J0 JST SH, J1 P3.5, J10 Pin Headers, J2 JST XH/PH, K1 Relay_SPDT, Q1 BSS138, SW0 SW_SPDT_MountingPin, SW1 Test Button

Commit message: Rename `connectors` symbol and footprint libraries to `connector`
Parts:
- J0: footprint connectors:JST_SH_SM03B-SRSS-TB_1x03-1MP_P1.00mm_Horizontal -> connector:JST_SH_SM03B-SRSS-TB_1x03-1MP_P1.00mm_Horizontal
Changed lines of the file:
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@@
 			)
 		)
-		(property "Footprint" "connectors:JST_SH_SM03B-SRSS-TB_1x03-1MP_P1.00mm_Horizontal"
+		(property "Footprint" "connector:JST_SH_SM03B-SRSS-TB_1x03-1MP_P1.00mm_Horizontal"
 			(at 207.01 92.71 0)
 			(effects
