File: pcb-archived/stackable1/relay-module-5v-x2/relay-module-5v-x2.kicad_sch (KiCad schematic)
At the start: 21 parts, among them J0 JST SH, J1 P5 or P3.5, J10 Pin Headers, J2 P5 or P3.5, K1 Relay_SPDT, K2 Relay_SPDT, Q1 2N7002DW, SW0 SW_SPDT_MountingPin, SW1 Test Button, SW2 Test Button

Commit message: Rename `connectors` symbol and footprint libraries to `connector`
Parts:
- J0: footprint connectors:JST_SH_SM04B-SRSS-TB_1x04-1MP_P1.00mm_Horizontal -> connector:JST_SH_SM04B-SRSS-TB_1x04-1MP_P1.00mm_Horizontal
Changed lines of the file:
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@@
 			)
 		)
-		(property "Footprint" "connectors:JST_SH_SM04B-SRSS-TB_1x04-1MP_P1.00mm_Horizontal"
+		(property "Footprint" "connector:JST_SH_SM04B-SRSS-TB_1x04-1MP_P1.00mm_Horizontal"
 			(at 209.55 100.33 0)
 			(effects
