File: pcb-archived/stackable1/esp-sensors/esp-sensors.kicad_sch (KiCad schematic)
At the start: 24 parts, among them J0 JST XH/PH, J1 JST SH, J2 JST SH, J3 JST SH, J4 JST SH, J5 JST SH, Q1 2N7002DW, Q2 BSS138, U1 TEMT6000X01

Commit message: Rename `connectors` symbol and footprint libraries to `connector`
Parts:
- J1, J2: footprint connectors:JST_SH_SM04B-SRSS-TB_1x04-1MP_P1.00mm_Horizontal -> connector:JST_SH_SM04B-SRSS-TB_1x04-1MP_P1.00mm_Horizontal
- J3: footprint connectors:JST_SH_SM03B-SRSS-TB_1x03-1MP_P1.00mm_Horizontal -> connector:JST_SH_SM03B-SRSS-TB_1x03-1MP_P1.00mm_Horizontal
- J4: footprint connectors:JST_SH_SM08B-SRSS-TB_1x08-1MP_P1.00mm_Horizontal -> connector:JST_SH_SM08B-SRSS-TB_1x08-1MP_P1.00mm_Horizontal
- J5: footprint connectors:JST_SH_SM06B-SRSS-TB_1x06-1MP_P1.00mm_Horizontal -> connector:JST_SH_SM06B-SRSS-TB_1x06-1MP_P1.00mm_Horizontal
Changed lines of the file:
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@@
 			)
 		)
-		(property "Footprint" "connectors:JST_SH_SM04B-SRSS-TB_1x04-1MP_P1.00mm_Horizontal"
+		(property "Footprint" "connector:JST_SH_SM04B-SRSS-TB_1x04-1MP_P1.00mm_Horizontal"
 			(at 142.24 27.94 0)
 			(effects
@@
 			)
 		)
-		(property "Footprint" "connectors:JST_SH_SM08B-SRSS-TB_1x08-1MP_P1.00mm_Horizontal"
+		(property "Footprint" "connector:JST_SH_SM08B-SRSS-TB_1x08-1MP_P1.00mm_Horizontal"
 			(at 180.34 25.4 0)
 			(effects
@@
 			)
 		)
-		(property "Footprint" "connectors:JST_SH_SM03B-SRSS-TB_1x03-1MP_P1.00mm_Horizontal"
+		(property "Footprint" "connector:JST_SH_SM03B-SRSS-TB_1x03-1MP_P1.00mm_Horizontal"
 			(at 111.76 53.34 0)
 			(effects
@@
 			)
 		)
-		(property "Footprint" "connectors:JST_SH_SM04B-SRSS-TB_1x04-1MP_P1.00mm_Horizontal"
+		(property "Footprint" "connector:JST_SH_SM04B-SRSS-TB_1x04-1MP_P1.00mm_Horizontal"
 			(at 142.24 50.8 0)
 			(effects
@@
 			)
 		)
-		(property "Footprint" "connectors:JST_SH_SM06B-SRSS-TB_1x06-1MP_P1.00mm_Horizontal"
+		(property "Footprint" "connector:JST_SH_SM06B-SRSS-TB_1x06-1MP_P1.00mm_Horizontal"
 			(at 173.99 50.8 0)
 			(effects

Commit message: Rename `modules` symbol and footprint libraries to `module`
Parts:
- SM1: footprint modules:ESP32-C3-Super-Mini-Castellated-SMD -> module:ESP32-C3-Super-Mini-Castellated-SMD; symbol modules:ESP32-C3-Super-Mini -> module:ESP32-C3-Super-Mini
- SM2: symbol modules:AHT20+BMP280 -> module:AHT20+BMP280
- SM3: symbol modules:ENS160+AHT2x -> module:ENS160+AHT2x
- SM4: symbol modules:BH1750 -> module:BH1750
Changed lines of the file:
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@@
 	)
 	(symbol
-		(lib_id "modules:ESP32-C3-Super-Mini")
+		(lib_id "module:ESP32-C3-Super-Mini")
 		(at 50.8 43.18 0)
 		(unit 1)
@@
 			)
 		)
-		(property "Footprint" "modules:ESP32-C3-Super-Mini-Castellated-SMD"
+		(property "Footprint" "module:ESP32-C3-Super-Mini-Castellated-SMD"
 			(at 50.8 43.18 0)
 			(effects
@@
 	)
 	(symbol
-		(lib_id "modules:ENS160+AHT2x")
+		(lib_id "module:ENS160+AHT2x")
 		(at 157.48 123.19 0)
 		(unit 1)
@@
 	)
 	(symbol
-		(lib_id "modules:BH1750")
+		(lib_id "module:BH1750")
 		(at 214.63 95.25 0)
 		(unit 1)
@@
 	)
 	(symbol
-		(lib_id "modules:AHT20+BMP280")
+		(lib_id "module:AHT20+BMP280")
 		(at 157.48 95.25 0)
 		(unit 1)
