File: pcb/stackable2/esp-cwww/esp-cwww.kicad_sch (KiCad schematic)
At the start: 37 parts, among them J0 Barrel_Jack_Switch, J1 JST PH, J2 Qwiic, Q1 ZC010DNG, Q2 BSS138, SW1 RotaryEncoder_Switch_MP, U1 TPS563200, U2 INA226

Commit message: Migrate `C_0402_1005Metric` footprint to `passives`
Parts:
- C10, C9: footprint custom:C_0402_1005Metric_simple -> passives:C_0402_1005Metric
Changed lines of the file:
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@@
 			)
 		)
-		(property "Footprint" "custom:C_0402_1005Metric_simple"
+		(property "Footprint" "passives:C_0402_1005Metric"
 			(at 262.89 97.79 0)
 			(effects
@@
 			)
 		)
-		(property "Footprint" "custom:C_0402_1005Metric_simple"
+		(property "Footprint" "passives:C_0402_1005Metric"
 			(at 217.17 97.79 0)
 			(effects

Commit message: Migrate `SOT-23` footprint to `packages`
Parts:
- Q2: footprint custom:SOT-23_simple -> packages:SOT-23
Changed lines of the file:
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@@
 			)
 		)
-		(property "Footprint" "custom:SOT-23_simple"
+		(property "Footprint" "packages:SOT-23"
 			(at 127.635 87.63 0)
 			(effects

Commit message: Migrate `PDFN-8_L3.2-W3.1-P0.65-LS3.4-BL-EP2` footprint to `packages`
Parts:
- Q1: footprint lcsc:PDFN-8_L3.2-W3.1-P0.65-LS3.4-BL-EP2 -> packages:PDFN-8_L3.2-W3.1-P0.65-LS3.4-BL-EP2
Changed lines of the file:
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@@
 			)
 		)
-		(property "Footprint" "lcsc:PDFN-8_L3.2-W3.1-P0.65-LS3.4-BL-EP2"
+		(property "Footprint" "packages:PDFN-8_L3.2-W3.1-P0.65-LS3.4-BL-EP2"
 			(at 60.96 106.045 0)
 			(effects
@@
 			)
 		)
-		(property "Footprint" "lcsc:PDFN-8_L3.2-W3.1-P0.65-LS3.4-BL-EP2"
+		(property "Footprint" "packages:PDFN-8_L3.2-W3.1-P0.65-LS3.4-BL-EP2"
 			(at 33.02 106.045 0)
 			(effects

Commit message: Migrate 2x2.5mm inductor footprint to `passives`
Parts:
- L1: footprint lcsc:IND-SMD_L2.5-W2.0_MHCHL2520 -> passives:L_1008_2520Metric_Molded
Changed lines of the file:
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@@
 			)
 		)
-		(property "Footprint" "lcsc:IND-SMD_L2.5-W2.0_MHCHL2520"
+		(property "Footprint" "passives:L_1008_2520Metric_Molded"
 			(at 170.18 30.48 0)
 			(effects

Commit message: Fix and update esp-cwww
Fixes:
- Fix SK6812SIDE pinout
- Add courtyard to SK6812SIDE footprint
- Swap WW/CW in GPIO and connector pinout

Updates:
- Update board info on silkscreen
- Use `packages` SOT-23-6 footprint for TPS563201
- Avoid thermal relief on DC barrel jack GND pad
- Modify shunt resistor value
- Update LCSC part numbers

Features:
- Add JST SH connector for optional external rotary encoder, with board
  edge inset
Parts:
- removed PIX1, PIX2: WS2812B-2020, lcsc:LED-SK6812SIDE-A-4x1.6mm, symbol LED:WS2812B-2020
- added J3: JST SH, connectors:JST_SH_SM05B-SRSS-TB_1x05-1MP_P1.00mm_Horizontal, symbol Connector_Generic_MountingPin:Conn_01x05_MountingPin
- added PIX1, PIX2: SK6812SIDE-A, lcsc:LED-SK6812SIDE-A-4x1.6mm, symbol lcsc:SK6812SIDE-A
- C10, C9: LCSC Part C1525 -> C152814
- R0: footprint Resistor_SMD:R_0603_1608Metric_Pad0.98x0.95mm_HandSolder -> passives:R_0402_1005Metric
- R6: LCSC Part (none) -> C25077
- SR1: value R040 -> R020; LCSC Part C2985725 -> C5375467
- U1: value TPS563200 -> TPS563201; footprint custom:SOT-23-6_Handsoldering_simple -> packages:SOT-23-6
Connections:
- net +3V3: now also J3.2 (Pin_2)
- net +5V: now also PIX1.2 (VDD), PIX2.2 (VDD)
- net BUTTON: now also J3.3 (Pin_3)
- net CLK: now also J3.5 (Pin_5)
- net CW_12V: now also J1.2 (Pin_2), J1.5 (Pin_5), Q1.5 (D); no longer J1.1 (Pin_1), J1.6 (Pin_6), Q1.6 (D)
- net CW_PWM_3V3: now also R4.2, SM1.1 (ADC/GPIO1); no longer R5.2, SM1.0 (ADC/GPIO0)
- net DT: now also J3.4 (Pin_4)
- net GND: now also J3.1 (Pin_1), J3.MP (MountPin), PIX1.4 (VSS), PIX2.4 (VSS)
- net NEOPIXEL_DATA_5V: now also PIX1.1 (DIN)
- net WW_12V: now also J1.1 (Pin_1), J1.6 (Pin_6), Q1.6 (D); no longer J1.2 (Pin_2), J1.5 (Pin_5), Q1.5 (D)
- net WW_PWM_3V3: now also R5.2, SM1.0 (ADC/GPIO0); no longer R4.2, SM1.1 (ADC/GPIO1)
- new net: PIX1.3 (DOUT), PIX2.1 (DIN)

Commit message: Rename `L_1008_2520Metric_Molded` to `L_1008_2520Metric`
Parts:
- L1: footprint passives:L_1008_2520Metric_Molded -> passives:L_1008_2520Metric
Changed lines of the file:
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@@
 			)
 		)
-		(property "Footprint" "passives:L_1008_2520Metric_Molded"
+		(property "Footprint" "passives:L_1008_2520Metric"
 			(at 170.18 30.48 0)
 			(effects

Commit message: Rename `connectors` symbol and footprint libraries to `connector`
Parts:
- J1: footprint connectors:JST_PH_S6B-PH-SM4-TB_1x06-1MP_P2.00mm_Horizontal -> connector:JST_PH_S6B-PH-SM4-TB_1x06-1MP_P2.00mm_Horizontal
- J2: footprint connectors:Qwiic-SMD-horizontal-logo -> connector:Qwiic-SMD-horizontal-logo; symbol connectors:Qwiic -> connector:Qwiic
- J3: footprint connectors:JST_SH_SM05B-SRSS-TB_1x05-1MP_P1.00mm_Horizontal -> connector:JST_SH_SM05B-SRSS-TB_1x05-1MP_P1.00mm_Horizontal
Changed lines of the file:
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@@
 	)
 	(symbol
-		(lib_id "connectors:Qwiic")
+		(lib_id "connector:Qwiic")
 		(at 92.71 160.02 0)
 		(unit 1)
@@
 			)
 		)
-		(property "Footprint" "connectors:Qwiic-SMD-horizontal-logo"
+		(property "Footprint" "connector:Qwiic-SMD-horizontal-logo"
 			(at 92.71 160.02 0)
 			(effects
@@
 			)
 		)
-		(property "Footprint" "connectors:JST_PH_S6B-PH-SM4-TB_1x06-1MP_P2.00mm_Horizontal"
+		(property "Footprint" "connector:JST_PH_S6B-PH-SM4-TB_1x06-1MP_P2.00mm_Horizontal"
 			(at 64.77 160.02 0)
 			(effects
@@
 			)
 		)
-		(property "Footprint" "connectors:JST_SH_SM05B-SRSS-TB_1x05-1MP_P1.00mm_Horizontal"
+		(property "Footprint" "connector:JST_SH_SM05B-SRSS-TB_1x05-1MP_P1.00mm_Horizontal"
 			(at 124.46 160.02 0)
 			(effects

Commit message: Rename `modules` symbol and footprint libraries to `module`
Parts:
- SM1: footprint modules:ESP32-C3-Super-Mini-Castellated-SMD-only -> module:ESP32-C3-Super-Mini-Castellated-SMD-only; symbol modules:ESP32-C3-Super-Mini -> module:ESP32-C3-Super-Mini
Changed lines of the file:
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@@
 	)
 	(symbol
-		(lib_id "modules:ESP32-C3-Super-Mini")
+		(lib_id "module:ESP32-C3-Super-Mini")
 		(at 49.53 36.83 0)
 		(unit 1)
@@
 			)
 		)
-		(property "Footprint" "modules:ESP32-C3-Super-Mini-Castellated-SMD-only"
+		(property "Footprint" "module:ESP32-C3-Super-Mini-Castellated-SMD-only"
 			(at 49.53 21.082 0)
 			(effects
