File: pcb/esphome/garage-door-control/garage-door-control.kicad_pcb (KiCad board)
At the start: 2 copper layers, 115 x 30 mm, 24 parts, among them J1 Barrel_Jack_Switch, J2 JST XH, J3 JST XH, J4 JST XH, K1 Relay_SPDT, Q1 BSS138, Q2 BSS138, Q3 BSS138, Q4 BSS138

Commit message: Migrate ESP32 module library references in projects
Parts:
- SM1: footprint aliexpress:ESP32-C3-Super-Mini-Pins -> modules:ESP32-C3-Super-Mini-Pins
Changed lines of the file:
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@@
 		)
 	)
-	(footprint "aliexpress:ESP32-C3-Super-Mini-Pins"
+	(footprint "modules:ESP32-C3-Super-Mini-Pins"
 		(layer "F.Cu")
 		(at 106.48 100.52 90)
@@
 			)
 		)
-		(property "Footprint" "aliexpress:ESP32-C3-Super-Mini-Pins"
+		(property "Footprint" "modules:ESP32-C3-Super-Mini-Pins"
 			(at 0 0 90)
 			(unlocked yes)
@@
 			(pintype "power_in")
 		)
-		(model "${KIPRJMOD}/libraries/aliexpress.3dshapes/ESP32-C3-SuperMini.step"
+		(model "${KIPRJMOD}/libraries/modules.3dshapes/ESP32-C3-SuperMini.step"
 			(offset
 				(xyz 0 -2.3 2.5)

Commit message: Migrate AHT20+BMP280 module library references in projects
Parts:
- SM2: footprint aliexpress:AHT20+BMP280-noholes -> modules:AHT20+BMP280-noholes
Changed lines of the file:
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@@
 		)
 	)
-	(footprint "aliexpress:AHT20+BMP280-noholes"
+	(footprint "modules:AHT20+BMP280-noholes"
 		(layer "F.Cu")
 		(at 145.938 95.4 -90)
@@
 			)
 		)
-		(property "Footprint" "aliexpress:AHT20+BMP280-noholes"
+		(property "Footprint" "modules:AHT20+BMP280-noholes"
 			(at 0 0 -90)
 			(unlocked yes)
@@
 			(pintype "input")
 		)
-		(model "${KIPRJMOD}/libraries/aliexpress.3dshapes/AHT20+BMP280.step"
+		(model "${KIPRJMOD}/libraries/modules.3dshapes/AHT20+BMP280.step"
 			(offset
 				(xyz -7.5 -7.5 4)

Commit message: Migrate ENS160+AHT2x module
Parts:
- SM3: footprint aliexpress:ENS160+AHT2x-noholes -> modules:ENS160+AHT2x-noholes
Changed lines of the file:
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@@
 		)
 	)
-	(footprint "aliexpress:ENS160+AHT2x-noholes"
+	(footprint "modules:ENS160+AHT2x-noholes"
 		(layer "F.Cu")
 		(at 165.02 99.9 -90)
@@
 			)
 		)
-		(property "Footprint" "aliexpress:ENS160+AHT2x-noholes"
+		(property "Footprint" "modules:ENS160+AHT2x-noholes"
 			(at 0 0 -90)
 			(unlocked yes)

Commit message: Migrate `D_SMA` footprint to `passives`
Parts:
- D1: footprint custom:D_SMA_simple -> passives:D_SMA
Changed lines of the file:
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@@
 		)
 	)
-	(footprint "custom:D_SMA_simple"
+	(footprint "passives:D_SMA"
 		(layer "F.Cu")
 		(at 200.6 101.9 -90)
@@
 			)
 		)
-		(property "Footprint" "custom:D_SMA_simple"
+		(property "Footprint" "passives:D_SMA"
 			(at 0 0 -90)
 			(unlocked yes)

Commit message: Migrate `D_SMA` footprint from `passives` to `packages`
Parts:
- D1: footprint passives:D_SMA -> packages:D_SMA
Changed lines of the file:
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@@
 		)
 	)
-	(footprint "passives:D_SMA"
+	(footprint "packages:D_SMA"
 		(layer "F.Cu")
 		(at 200.6 101.9 -90)
@@
 			)
 		)
-		(property "Footprint" "passives:D_SMA"
+		(property "Footprint" "packages:D_SMA"
 			(at 0 0 -90)
 			(unlocked yes)

Commit message: Rename `modules` symbol and footprint libraries to `module`
Parts:
- SM1: footprint modules:ESP32-C3-Super-Mini-Pins -> module:ESP32-C3-Super-Mini-Pins
- SM2: footprint modules:AHT20+BMP280-noholes -> module:AHT20+BMP280-noholes
- SM3: footprint modules:ENS160+AHT2x-noholes -> module:ENS160+AHT2x-noholes
Changed lines of the file:
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@@
 		)
 	)
-	(footprint "modules:AHT20+BMP280-noholes"
+	(footprint "module:AHT20+BMP280-noholes"
 		(layer "F.Cu")
 		(at 145.938 95.4 -90)
@@
 			)
 		)
-		(property "Footprint" "modules:AHT20+BMP280-noholes"
+		(property "Footprint" "module:AHT20+BMP280-noholes"
 			(at 0 0 -90)
 			(unlocked yes)
@@
 			(pintype "input")
 		)
-		(model "${KIPRJMOD}/libraries/modules.3dshapes/AHT20+BMP280.step"
+		(model "${KIPRJMOD}/libraries/module.3dshapes/AHT20+BMP280.step"
 			(offset
 				(xyz -7.5 -7.5 4)
@@
 		)
 	)
-	(footprint "modules:ENS160+AHT2x-noholes"
+	(footprint "module:ENS160+AHT2x-noholes"
 		(layer "F.Cu")
 		(at 165.02 99.9 -90)
@@
 			)
 		)
-		(property "Footprint" "modules:ENS160+AHT2x-noholes"
+		(property "Footprint" "module:ENS160+AHT2x-noholes"
 			(at 0 0 -90)
 			(unlocked yes)
@@
 		)
 	)
-	(footprint "modules:ESP32-C3-Super-Mini-Pins"
+	(footprint "module:ESP32-C3-Super-Mini-Pins"
 		(layer "F.Cu")
 		(at 106.48 100.52 90)
@@
 			)
 		)
-		(property "Footprint" "modules:ESP32-C3-Super-Mini-Pins"
+		(property "Footprint" "module:ESP32-C3-Super-Mini-Pins"
 			(at 0 0 90)
 			(unlocked yes)
@@
 			(pintype "power_in")
 		)
-		(model "${KIPRJMOD}/libraries/modules.3dshapes/ESP32-C3-SuperMini.step"
+		(model "${KIPRJMOD}/libraries/module.3dshapes/ESP32-C3-SuperMini.step"
 			(offset
 				(xyz 0 -2.3 2.5)

Commit message: Rename `packages` footprint library to `package`
Parts:
- D1: footprint packages:D_SMA -> package:D_SMA
Changed lines of the file:
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@@
 		)
 	)
-	(footprint "packages:D_SMA"
+	(footprint "package:D_SMA"
 		(layer "F.Cu")
 		(at 200.6 101.9 -90)
@@
 			)
 		)
-		(property "Footprint" "packages:D_SMA"
+		(property "Footprint" "package:D_SMA"
 			(at 0 0 -90)
 			(unlocked yes)

Commit message: Rework `ENS160+AHT2x` symbol to match KiCAD symbol conventions
Parts:
- SM2: value ~ -> AHT20+BMP280
- SM3: value ~ -> ENS160+AHT2x
Changed lines of the file:
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@@
 			)
 		)
-		(property "Value" "~"
+		(property "Value" "AHT20+BMP280"
 			(at 0 1 -90)
 			(unlocked yes)
@@
 			)
 		)
-		(property "Datasheet" ""
+		(property "Datasheet" "https://cdn-learn.adafruit.com/assets/assets/000/123/394/original/Data_Sheet_AHT20.pdf?1691532479"
 			(at 0 0 -90)
 			(unlocked yes)
@@
 			)
 		)
-		(property "Description" ""
+		(property "Description" "Combination Digital Temperature, Absolute Barometric Pressure Sensor module"
 			(at 0 0 -90)
 			(unlocked yes)
@@
 				(font
 					(size 1.27 1.27)
+					(thickness 0.15)
+				)
+			)
+		)
+		(property "Datasheet2" "https://ae-bst.resource.bosch.com/media/_tech/media/datasheets/BST-BMP280-DS001.pdf"
+			(at 0 0 -90)
+			(unlocked yes)
+			(layer "F.Fab")
+			(hide yes)
+			(effects
+				(font
+					(size 1 1)
 					(thickness 0.15)
 				)
@@
 			)
 		)
-		(property "Value" "~"
+		(property "Value" "ENS160+AHT2x"
 			(at -1.524 -7.62 -90)
 			(unlocked yes)
@@
 			)
 		)
-		(property "Datasheet" ""
+		(property "Datasheet" "https://www.sciosense.com/wp-content/uploads/2023/12/ENS160-Datasheet.pdf"
 			(at 0 0 -90)
 			(unlocked yes)
@@
 			)
 		)
-		(property "Description" ""
+		(property "Description" "Combination Air Quality, Digital Temperature Sensor module"
 			(at 0 0 -90)
 			(unlocked yes)
@@
 				(font
 					(size 1.27 1.27)
+					(thickness 0.15)
+				)
+			)
+		)
+		(property "Datasheet2" "https://cdn-learn.adafruit.com/assets/assets/000/123/394/original/Data_Sheet_AHT20.pdf?1691532479"
+			(at 0 0 -90)
+			(unlocked yes)
+			(layer "F.Fab")
+			(hide yes)
+			(effects
+				(font
+					(size 1 1)
 					(thickness 0.15)
 				)
@@
 			)
 		)
+		(fp_text user "SCL/SCLK"
+			(at -1.27 6.75 180)
+			(unlocked yes)
+			(layer "B.SilkS")
+			(effects
+				(font
+					(size 0.7 0.7)
+					(thickness 0.1)
+				)
+				(justify left mirror)
+			)
+		)
+		(fp_text user "SDA/MOSI"
+			(at 1.27 6.75 180)
+			(unlocked yes)
+			(layer "B.SilkS")
+			(effects
+				(font
+					(size 0.7 0.7)
+					(thickness 0.1)
+				)
+				(justify left mirror)
+			)
+		)
+		(fp_text user "CS"
+			(at 6.35 6.75 180)
+			(unlocked yes)
+			(layer "B.SilkS")
+			(effects
+				(font
+					(size 0.7 0.7)
+					(thickness 0.1)
+				)
+				(justify left mirror)
+			)
+		)
+		(fp_text user "GND"
+			(at -3.81 6.75 180)
+			(unlocked yes)
+			(layer "B.SilkS")
+			(effects
+				(font
+					(size 0.7 0.7)
+					(thickness 0.1)
+				)
+				(justify left mirror)
+			)
+		)
 		(fp_text user "ADD/MISO"
 			(at 3.81 6.75 180)
@@
 			)
 		)
-		(fp_text user "CS"
-			(at 6.35 6.75 180)
-			(unlocked yes)
-			(layer "B.SilkS")
-			(effects
-				(font
-					(size 0.7 0.7)
-					(thickness 0.1)
-				)
-				(justify left mirror)
-			)
-		)
-		(fp_text user "SCL/SCLK"
-			(at -1.27 6.75 180)
-			(unlocked yes)
-			(layer "B.SilkS")
-			(effects
-				(font
-					(size 0.7 0.7)
-					(thickness 0.1)
-				)
-				(justify left mirror)
-			)
-		)
-		(fp_text user "SDA/MOSI"
-			(at 1.27 6.75 180)
-			(unlocked yes)
-			(layer "B.SilkS")
-			(effects
-				(font
-					(size 0.7 0.7)
-					(thickness 0.1)
-				)
-				(justify left mirror)
-			)
-		)
-		(fp_text user "GND"
-			(at -3.81 6.75 180)
-			(unlocked yes)
-			(layer "B.SilkS")
-			(effects
-				(font
-					(size 0.7 0.7)
-					(thickness 0.1)
-				)
-				(justify left mirror)
-			)
-		)
 		(fp_text user "VIN"
 			(at -8.89 6.75 180)
@@
 			)
 		)
+		(fp_text user "ADD"
+			(at 3.81 6.75 -90)
+			(unlocked yes)
+			(layer "F.SilkS")
+			(effects
+				(font
+					(size 0.7 0.7)
+					(thickness 0.1)
+				)
+				(justify bottom)
+			)
+		)
+		(fp_text user "VIN"
+			(at -8.89 6.75 -90)
+			(unlocked yes)
+			(layer "F.SilkS")
+			(effects
+				(font
+					(size 0.7 0.7)
+					(thickness 0.1)
+				)
+				(justify bottom)
+			)
+		)
+		(fp_text user "3V3"
+			(at -6.35 6.75 -90)
+			(unlocked yes)
+			(layer "F.SilkS")
+			(effects
+				(font
+					(size 0.7 0.7)
+					(thickness 0.1)
+				)
+				(justify bottom)
+			)
+		)
+		(fp_text user "INT"
+			(at 8.89 6.75 -90)
+			(unlocked yes)
+			(layer "F.SilkS")
+			(effects
+				(font
+					(size 0.7 0.7)
+					(thickness 0.1)
+				)
+				(justify bottom)
+			)
+		)
+		(fp_text user "ENS160+AHT2x"
+			(at 0 0 -90)
+			(unlocked yes)
+			(layer "F.SilkS")
+			(effects
+				(font
+					(size 1 1)
+					(thickness 0.15)
+				)
+			)
+		)
 		(fp_text user "SCL"
 			(at -1.27 6.75 -90)
@@
 			)
 		)
-		(fp_text user "ENS160+AHT2x"
-			(at 0 0 -90)
-			(unlocked yes)
-			(layer "F.SilkS")
-			(effects
-				(font
-					(size 1 1)
-					(thickness 0.15)
-				)
+		(fp_text user "CS"
+			(at 6.35 6.75 -90)
+			(unlocked yes)
+			(layer "F.SilkS")
+			(effects
+				(font
+					(size 0.7 0.7)
+					(thickness 0.1)
+				)
+				(justify bottom)
 			)
 		)
@@
 			)
 		)
-		(fp_text user "CS"
-			(at 6.35 6.75 -90)
-			(unlocked yes)
-			(layer "F.SilkS")
-			(effects
-				(font
-					(size 0.7 0.7)
-					(thickness 0.1)
-				)
-				(justify bottom)
-			)
-		)
-		(fp_text user "ADD"
-			(at 3.81 6.75 -90)
-			(unlocked yes)
-			(layer "F.SilkS")
-			(effects
-				(font
-					(size 0.7 0.7)
-					(thickness 0.1)
-				)
-				(justify bottom)
-			)
-		)
-		(fp_text user "VIN"
-			(at -8.89 6.75 -90)
-			(unlocked yes)
-			(layer "F.SilkS")
-			(effects
-				(font
-					(size 0.7 0.7)
-					(thickness 0.1)
-				)
-				(justify bottom)
-			)
-		)
-		(fp_text user "3V3"
-			(at -6.35 6.75 -90)
-			(unlocked yes)
-			(layer "F.SilkS")
-			(effects
-				(font
-					(size 0.7 0.7)
-					(thickness 0.1)
-				)
-				(justify bottom)
-			)
-		)
 		(fp_text user "SDA"
 			(at 1.27 6.75 -90)
 			(unlocked yes)
 			(layer "F.SilkS")
-			(effects
-				(font
-					(size 0.7 0.7)
-					(thickness 0.1)
-				)
-				(justify bottom)
-			)
-		)
-		(fp_text user "INT"
-			(at 8.89 6.75 -90)
-			(unlocked yes)
-			(layer "F.SilkS")
