File: pcb/misc/gr6408/gr6408.kicad_sch (KiCad schematic)
At the start: 39 parts, among them J1 Pin headers, J2 Pin headers, Q1 AO3400A, Q2 AO3400A, U1 GR6408

Commit message: Migrate `C_0603_1608Metric` footprint to `passives`
Parts:
- C1: footprint custom:C_0603_1608Metric -> passives:C_0603_1608Metric
Changed lines of the file:
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@@
 			)
 		)
-		(property "Footprint" "custom:C_0603_1608Metric"
+		(property "Footprint" "passives:C_0603_1608Metric"
 			(at 137.16 34.29 0)
 			(effects

Commit message: Migrate `R_0603_1608Metric` footprint to `passives`
Parts:
- R1, R2, R3, R4, R5, R6, R7, R8, R9: footprint custom:R_0603_1608Metric_simple -> passives:R_0603_1608Metric
Changed lines of the file:
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@@
 			)
 		)
-		(property "Footprint" "custom:R_0603_1608Metric_simple"
+		(property "Footprint" "passives:R_0603_1608Metric"
 			(at 201.93 68.58 0)
 			(effects
@@
 			)
 		)
-		(property "Footprint" "custom:R_0603_1608Metric_simple"
+		(property "Footprint" "passives:R_0603_1608Metric"
 			(at 198.12 60.96 0)
 			(effects
@@
 			)
 		)
-		(property "Footprint" "custom:R_0603_1608Metric_simple"
+		(property "Footprint" "passives:R_0603_1608Metric"
 			(at 172.72 77.47 0)
 			(effects
@@
 			)
 		)
-		(property "Footprint" "custom:R_0603_1608Metric_simple"
+		(property "Footprint" "passives:R_0603_1608Metric"
 			(at 213.36 60.96 0)
 			(effects
@@
 			)
 		)
-		(property "Footprint" "custom:R_0603_1608Metric_simple"
+		(property "Footprint" "passives:R_0603_1608Metric"
 			(at 217.17 68.58 0)
 			(effects
@@
 			)
 		)
-		(property "Footprint" "custom:R_0603_1608Metric_simple"
+		(property "Footprint" "passives:R_0603_1608Metric"
 			(at 77.47 97.79 0)
 			(effects
@@
 			)
 		)
-		(property "Footprint" "custom:R_0603_1608Metric_simple"
+		(property "Footprint" "passives:R_0603_1608Metric"
 			(at 209.55 68.58 0)
 			(effects
@@
 			)
 		)
-		(property "Footprint" "custom:R_0603_1608Metric_simple"
+		(property "Footprint" "passives:R_0603_1608Metric"
 			(at 172.72 67.31 0)
 			(effects
@@
 			)
 		)
-		(property "Footprint" "custom:R_0603_1608Metric_simple"
+		(property "Footprint" "passives:R_0603_1608Metric"
 			(at 194.31 68.58 0)
 			(effects

Commit message: Migrate `LED_0402_1005Metric` footprint to `passives`
Parts:
- LED1, LED10, LED11, LED12, LED13, LED14, LED15, LED16, LED2, LED3, LED4, LED5, LED6, LED7, LED8, LED9: footprint custom:LED_0402_1005Metric -> passives:LED_0402_1005Metric
Changed lines of the file:
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@@
 			)
 		)
-		(property "Footprint" "custom:LED_0402_1005Metric"
+		(property "Footprint" "passives:LED_0402_1005Metric"
 			(at 195.58 153.67 90)
 			(effects
@@
 			)
 		)
-		(property "Footprint" "custom:LED_0402_1005Metric"
+		(property "Footprint" "passives:LED_0402_1005Metric"
 			(at 149.86 104.14 90)
 			(effects
@@
 			)
 		)
-		(property "Footprint" "custom:LED_0402_1005Metric"
+		(property "Footprint" "passives:LED_0402_1005Metric"
 			(at 180.34 153.67 90)
 			(effects
@@
 			)
 		)
-		(property "Footprint" "custom:LED_0402_1005Metric"
+		(property "Footprint" "passives:LED_0402_1005Metric"
 			(at 104.14 153.67 90)
 			(effects
@@
 			)
 		)
-		(property "Footprint" "custom:LED_0402_1005Metric"
+		(property "Footprint" "passives:LED_0402_1005Metric"
 			(at 134.62 153.67 90)
 			(effects
@@
 			)
 		)
-		(property "Footprint" "custom:LED_0402_1005Metric"
+		(property "Footprint" "passives:LED_0402_1005Metric"
 			(at 195.58 104.14 90)
 			(effects
@@
 			)
 		)
-		(property "Footprint" "custom:LED_0402_1005Metric"
+		(property "Footprint" "passives:LED_0402_1005Metric"
 			(at 165.1 153.67 90)
 			(effects
@@
 			)
 		)
-		(property "Footprint" "custom:LED_0402_1005Metric"
+		(property "Footprint" "passives:LED_0402_1005Metric"
 			(at 119.38 104.14 90)
 			(effects
@@
 			)
 		)
-		(property "Footprint" "custom:LED_0402_1005Metric"
+		(property "Footprint" "passives:LED_0402_1005Metric"
 			(at 88.9 153.67 90)
 			(effects
@@
 			)
 		)
-		(property "Footprint" "custom:LED_0402_1005Metric"
+		(property "Footprint" "passives:LED_0402_1005Metric"
 			(at 134.62 104.14 90)
 			(effects
@@
 			)
 		)
-		(property "Footprint" "custom:LED_0402_1005Metric"
+		(property "Footprint" "passives:LED_0402_1005Metric"
 			(at 180.34 104.14 90)
 			(effects
@@
 			)
 		)
-		(property "Footprint" "custom:LED_0402_1005Metric"
+		(property "Footprint" "passives:LED_0402_1005Metric"
 			(at 88.9 104.14 90)
 			(effects
@@
 			)
 		)
-		(property "Footprint" "custom:LED_0402_1005Metric"
+		(property "Footprint" "passives:LED_0402_1005Metric"
 			(at 104.14 104.14 90)
 			(effects
@@
 			)
 		)
-		(property "Footprint" "custom:LED_0402_1005Metric"
+		(property "Footprint" "passives:LED_0402_1005Metric"
 			(at 165.1 104.14 90)
 			(effects
@@
 			)
 		)
-		(property "Footprint" "custom:LED_0402_1005Metric"
+		(property "Footprint" "passives:LED_0402_1005Metric"
 			(at 149.86 153.67 90)
 			(effects
@@
 			)
 		)
-		(property "Footprint" "custom:LED_0402_1005Metric"
+		(property "Footprint" "passives:LED_0402_1005Metric"
 			(at 119.38 153.67 90)
 			(effects

Commit message: Migrate `LED_0402_1005Metric` footprint to `led`
Parts:
- LED1, LED10, LED11, LED12, LED13, LED14, LED15, LED16, LED2, LED3, LED4, LED5, LED6, LED7, LED8, LED9: footprint passives:LED_0402_1005Metric -> led:LED_0402_1005Metric
Changed lines of the file:
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@@
 			)
 		)
-		(property "Footprint" "passives:LED_0402_1005Metric"
+		(property "Footprint" "led:LED_0402_1005Metric"
 			(at 195.58 153.67 90)
 			(effects
@@
 			)
 		)
-		(property "Footprint" "passives:LED_0402_1005Metric"
+		(property "Footprint" "led:LED_0402_1005Metric"
 			(at 149.86 104.14 90)
 			(effects
@@
 			)
 		)
-		(property "Footprint" "passives:LED_0402_1005Metric"
+		(property "Footprint" "led:LED_0402_1005Metric"
 			(at 180.34 153.67 90)
 			(effects
@@
 			)
 		)
-		(property "Footprint" "passives:LED_0402_1005Metric"
+		(property "Footprint" "led:LED_0402_1005Metric"
 			(at 104.14 153.67 90)
 			(effects
@@
 			)
 		)
-		(property "Footprint" "passives:LED_0402_1005Metric"
+		(property "Footprint" "led:LED_0402_1005Metric"
 			(at 134.62 153.67 90)
 			(effects
@@
 			)
 		)
-		(property "Footprint" "passives:LED_0402_1005Metric"
+		(property "Footprint" "led:LED_0402_1005Metric"
 			(at 195.58 104.14 90)
 			(effects
@@
 			)
 		)
-		(property "Footprint" "passives:LED_0402_1005Metric"
+		(property "Footprint" "led:LED_0402_1005Metric"
 			(at 165.1 153.67 90)
 			(effects
@@
 			)
 		)
-		(property "Footprint" "passives:LED_0402_1005Metric"
+		(property "Footprint" "led:LED_0402_1005Metric"
 			(at 119.38 104.14 90)
 			(effects
@@
 			)
 		)
-		(property "Footprint" "passives:LED_0402_1005Metric"
+		(property "Footprint" "led:LED_0402_1005Metric"
 			(at 88.9 153.67 90)
 			(effects
@@
 			)
 		)
-		(property "Footprint" "passives:LED_0402_1005Metric"
+		(property "Footprint" "led:LED_0402_1005Metric"
 			(at 134.62 104.14 90)
 			(effects
@@
 			)
 		)
-		(property "Footprint" "passives:LED_0402_1005Metric"
+		(property "Footprint" "led:LED_0402_1005Metric"
 			(at 180.34 104.14 90)
 			(effects
@@
 			)
 		)
-		(property "Footprint" "passives:LED_0402_1005Metric"
+		(property "Footprint" "led:LED_0402_1005Metric"
 			(at 88.9 104.14 90)
 			(effects
@@
 			)
 		)
-		(property "Footprint" "passives:LED_0402_1005Metric"
+		(property "Footprint" "led:LED_0402_1005Metric"
 			(at 104.14 104.14 90)
 			(effects
@@
 			)
 		)
-		(property "Footprint" "passives:LED_0402_1005Metric"
+		(property "Footprint" "led:LED_0402_1005Metric"
 			(at 165.1 104.14 90)
 			(effects
@@
 			)
 		)
-		(property "Footprint" "passives:LED_0402_1005Metric"
+		(property "Footprint" "led:LED_0402_1005Metric"
 			(at 149.86 153.67 90)
 			(effects
@@
 			)
 		)
-		(property "Footprint" "passives:LED_0402_1005Metric"
+		(property "Footprint" "led:LED_0402_1005Metric"
 			(at 119.38 153.67 90)
 			(effects

Commit message: Rename `passives` footprint library to `passive`
Parts:
- C1: footprint passives:C_0603_1608Metric -> passive:C_0603_1608Metric
- R1, R2, R3, R4, R5, R6, R7, R8, R9: footprint passives:R_0603_1608Metric -> passive:R_0603_1608Metric
Changed lines of the file:
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@@
 			)
 		)
-		(property "Footprint" "passives:R_0603_1608Metric"
+		(property "Footprint" "passive:R_0603_1608Metric"
 			(at 201.93 68.58 0)
 			(effects
@@
 			)
 		)
-		(property "Footprint" "passives:R_0603_1608Metric"
+		(property "Footprint" "passive:R_0603_1608Metric"
 			(at 198.12 60.96 0)
 			(effects
@@
 			)
 		)
-		(property "Footprint" "passives:C_0603_1608Metric"
+		(property "Footprint" "passive:C_0603_1608Metric"
 			(at 137.16 34.29 0)
 			(effects
@@
 			)
 		)
-		(property "Footprint" "passives:R_0603_1608Metric"
+		(property "Footprint" "passive:R_0603_1608Metric"
 			(at 172.72 77.47 0)
 			(effects
@@
 			)
 		)
-		(property "Footprint" "passives:R_0603_1608Metric"
+		(property "Footprint" "passive:R_0603_1608Metric"
 			(at 213.36 60.96 0)
 			(effects
@@
 			)
 		)
-		(property "Footprint" "passives:R_0603_1608Metric"
+		(property "Footprint" "passive:R_0603_1608Metric"
 			(at 217.17 68.58 0)
 			(effects
@@
 			)
 		)
-		(property "Footprint" "passives:R_0603_1608Metric"
+		(property "Footprint" "passive:R_0603_1608Metric"
 			(at 77.47 97.79 0)
 			(effects
@@
 			)
 		)
-		(property "Footprint" "passives:R_0603_1608Metric"
+		(property "Footprint" "passive:R_0603_1608Metric"
 			(at 209.55 68.58 0)
 			(effects
@@
 			)
 		)
-		(property "Footprint" "passives:R_0603_1608Metric"
+		(property "Footprint" "passive:R_0603_1608Metric"
 			(at 172.72 67.31 0)
 			(effects
@@
 			)
 		)
-		(property "Footprint" "passives:R_0603_1608Metric"
+		(property "Footprint" "passive:R_0603_1608Metric"
 			(at 194.31 68.58 0)
 			(effects

Commit message: Rename `passive` footprint library to `discrete`
Parts:
- C1: footprint passive:C_0603_1608Metric -> discrete:C_0603_1608Metric
- R1, R2, R3, R4, R5, R6, R7, R8, R9: footprint passive:R_0603_1608Metric -> discrete:R_0603_1608Metric
Changed lines of the file:
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@@
 			)
 		)
-		(property "Footprint" "passive:R_0603_1608Metric"
+		(property "Footprint" "discrete:R_0603_1608Metric"
 			(at 201.93 68.58 0)
 			(effects
@@
 			)
 		)
-		(property "Footprint" "passive:R_0603_1608Metric"
+		(property "Footprint" "discrete:R_0603_1608Metric"
 			(at 198.12 60.96 0)
 			(effects
@@
 			)
 		)
-		(property "Footprint" "passive:C_0603_1608Metric"
+		(property "Footprint" "discrete:C_0603_1608Metric"
 			(at 137.16 34.29 0)
 			(effects
@@
 			)
 		)
-		(property "Footprint" "passive:R_0603_1608Metric"
+		(property "Footprint" "discrete:R_0603_1608Metric"
 			(at 172.72 77.47 0)
 			(effects
@@
 			)
 		)
-		(property "Footprint" "passive:R_0603_1608Metric"
+		(property "Footprint" "discrete:R_0603_1608Metric"
 			(at 213.36 60.96 0)
 			(effects
@@
 			)
 		)
-		(property "Footprint" "passive:R_0603_1608Metric"
+		(property "Footprint" "discrete:R_0603_1608Metric"
 			(at 217.17 68.58 0)
 			(effects
@@
 			)
 		)
-		(property "Footprint" "passive:R_0603_1608Metric"
+		(property "Footprint" "discrete:R_0603_1608Metric"
 			(at 77.47 97.79 0)
 			(effects
@@
 			)
 		)
-		(property "Footprint" "passive:R_0603_1608Metric"
+		(property "Footprint" "discrete:R_0603_1608Metric"
 			(at 209.55 68.58 0)
 			(effects
@@
 			)
 		)
-		(property "Footprint" "passive:R_0603_1608Metric"
+		(property "Footprint" "discrete:R_0603_1608Metric"
 			(at 172.72 67.31 0)
 			(effects
@@
 			)
 		)
-		(property "Footprint" "passive:R_0603_1608Metric"
+		(property "Footprint" "discrete:R_0603_1608Metric"
 			(at 194.31 68.58 0)
 			(effects

Commit message: Migrate `GR6408` symbol from `lcsc` to `ic`
Parts:
- U1: symbol lcsc:GR6408 -> ic:GR6408
Changed lines of the file:
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@@
 	)
 	(symbol
-		(lib_id "lcsc:GR6408")
+		(lib_id "ic:GR6408")
 		(at 149.86 57.15 0)
 		(unit 1)

Commit message: Migrate `LED_0402_1005Metric` from `led` to `discrete`
Parts:
- LED1, LED10, LED11, LED12, LED13, LED14, LED15, LED16, LED2, LED3, LED4, LED5, LED6, LED7, LED8, LED9: footprint led:LED_0402_1005Metric -> discrete:LED_0402_1005Metric
Changed lines of the file:
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@@
 			)
 		)
-		(property "Footprint" "led:LED_0402_1005Metric"
+		(property "Footprint" "discrete:LED_0402_1005Metric"
 			(at 195.58 153.67 90)
 			(effects
@@
 			)
 		)
-		(property "Footprint" "led:LED_0402_1005Metric"
+		(property "Footprint" "discrete:LED_0402_1005Metric"
 			(at 149.86 104.14 90)
 			(effects
@@
 			)
 		)
-		(property "Footprint" "led:LED_0402_1005Metric"
+		(property "Footprint" "discrete:LED_0402_1005Metric"
 			(at 180.34 153.67 90)
 			(effects
@@
 			)
 		)
-		(property "Footprint" "led:LED_0402_1005Metric"
+		(property "Footprint" "discrete:LED_0402_1005Metric"
 			(at 104.14 153.67 90)
 			(effects
@@
 			)
 		)
-		(property "Footprint" "led:LED_0402_1005Metric"
+		(property "Footprint" "discrete:LED_0402_1005Metric"
 			(at 134.62 153.67 90)
 			(effects
@@
 			)
 		)
-		(property "Footprint" "led:LED_0402_1005Metric"
+		(property "Footprint" "discrete:LED_0402_1005Metric"
 			(at 195.58 104.14 90)
 			(effects
@@
 			)
 		)
-		(property "Footprint" "led:LED_0402_1005Metric"
+		(property "Footprint" "discrete:LED_0402_1005Metric"
 			(at 165.1 153.67 90)
 			(effects
@@
 			)
 		)
-		(property "Footprint" "led:LED_0402_1005Metric"
+		(property "Footprint" "discrete:LED_0402_1005Metric"
 			(at 119.38 104.14 90)
 			(effects
@@
 			)
 		)
-		(property "Footprint" "led:LED_0402_1005Metric"
+		(property "Footprint" "discrete:LED_0402_1005Metric"
 			(at 88.9 153.67 90)
 			(effects
@@
 			)
 		)
-		(property "Footprint" "led:LED_0402_1005Metric"
+		(property "Footprint" "discrete:LED_0402_1005Metric"
 			(at 134.62 104.14 90)
 			(effects
@@
 			)
 		)
-		(property "Footprint" "led:LED_0402_1005Metric"
+		(property "Footprint" "discrete:LED_0402_1005Metric"
 			(at 180.34 104.14 90)
 			(effects
@@
 			)
 		)
-		(property "Footprint" "led:LED_0402_1005Metric"
+		(property "Footprint" "discrete:LED_0402_1005Metric"
 			(at 88.9 104.14 90)
 			(effects
@@
 			)
 		)
-		(property "Footprint" "led:LED_0402_1005Metric"
+		(property "Footprint" "discrete:LED_0402_1005Metric"
 			(at 104.14 104.14 90)
 			(effects
@@
 			)
 		)
-		(property "Footprint" "led:LED_0402_1005Metric"
+		(property "Footprint" "discrete:LED_0402_1005Metric"
 			(at 165.1 104.14 90)
 			(effects
@@
 			)
 		)
-		(property "Footprint" "led:LED_0402_1005Metric"
+		(property "Footprint" "discrete:LED_0402_1005Metric"
 			(at 149.86 153.67 90)
 			(effects
@@
 			)
 		)
-		(property "Footprint" "led:LED_0402_1005Metric"
+		(property "Footprint" "discrete:LED_0402_1005Metric"
 			(at 119.38 153.67 90)
 			(effects
