File: pcb/jigs/led-micro/led-micro.kicad_sch (KiCad schematic)
At the start: 13 parts, among them J1 Conn_01x04, J2 Conn_01x04

Commit message: Migrate `XL-2012RGBC` symbol from `lcsc` to `discrete`
Parts:
- LED0: symbol lcsc:XL-2012RGBC -> discrete:XL-2012RGBC
Changed lines of the file:
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@@
 	)
 	(symbol
-		(lib_id "lcsc:XL-2012RGBC")
+		(lib_id "discrete:XL-2012RGBC")
 		(at 154.94 130.81 0)
 		(mirror y)

Commit message: Rework XL-2012RGBC footprints, migrate from `lcsc` to `discrete`
Parts:
- LED0: footprint lcsc:LED-ARRAY-SMD_4P-L2.0-W1.3-BR_HandSolder -> discrete:LED_RGB_XL-2012RGBC_2.0x1.2mm_HandSolder
Changed lines of the file:
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@@
 			)
 		)
-		(property "Footprint" "lcsc:LED-ARRAY-SMD_4P-L2.0-W1.3-BR_HandSolder"
+		(property "Footprint" "discrete:LED_RGB_XL-2012RGBC_2.0x1.2mm_HandSolder"
 			(at 154.94 132.08 0)
 			(effects
