File: pcb/jigs/led-micro/led-micro.kicad_pcb (KiCad board)
At the start: 2 copper layers, 13 x 10.5 mm, 15 parts, among them J1 Conn_01x04, J2 Conn_01x04

Commit message: Rework XL-2012RGBC footprints, migrate from `lcsc` to `discrete`
Parts:
- LED0: footprint lcsc:LED-ARRAY-SMD_4P-L2.0-W1.3-BR_HandSolder -> discrete:LED_RGB_XL-2012RGBC_2.0x1.2mm_HandSolder
Changed lines of the file:
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@@
 		(property ki_fp_filters "DIP* SOIC* R*Array*Concave* R*Array*Convex* MSOP*")
 		(sheetname "Root")
-		(sheetfile "led-jig-mini.kicad_sch")
+		(sheetfile "led-micro.kicad_sch")
 		(attr smd)
 		(fp_line
@@
 		(property ki_fp_filters "LED* LED_SMD:* LED_THT:*")
 		(sheetname "Root")
-		(sheetfile "led-jig-mini.kicad_sch")
+		(sheetfile "led-micro.kicad_sch")
 		(attr smd)
 		(fp_poly
@@
 		(property ki_fp_filters "LED* LED_SMD:* LED_THT:*")
 		(sheetname "Root")
-		(sheetfile "led-jig-mini.kicad_sch")
+		(sheetfile "led-micro.kicad_sch")
 		(attr smd)
 		(fp_poly
@@
 		(property ki_fp_filters "LED* LED_SMD:* LED_THT:*")
 		(sheetname "Root")
-		(sheetfile "led-jig-mini.kicad_sch")
+		(sheetfile "led-micro.kicad_sch")
 		(attr smd)
 		(fp_poly
@@
 		(property ki_fp_filters "LED* LED_SMD:* LED_THT:*")
 		(sheetname "Root")
-		(sheetfile "led-jig-mini.kicad_sch")
+		(sheetfile "led-micro.kicad_sch")
 		(attr smd)
 		(fp_poly
@@
 		(property ki_fp_filters "SolderJumper*Open*")
 		(sheetname "Root")
-		(sheetfile "led-jig-mini.kicad_sch")
+		(sheetfile "led-micro.kicad_sch")
 		(zone_connect 1)
 		(attr exclude_from_pos_files exclude_from_bom)
@@
 		)
 	)
-	(footprint "lcsc:LED-ARRAY-SMD_4P-L2.0-W1.3-BR_HandSolder"
+	(footprint "discrete:LED_RGB_XL-2012RGBC_2.0x1.2mm_HandSolder"
 		(layer "F.Cu")
 		(at 134.075 99.06 180)
 		(property "Reference" "LED0"
-			(at 0 -2 0)
+			(at 0 -2 180)
 			(layer "Dwgs.User")
-			(hide yes)
 			(effects
 				(font
@@
 		)
 		(property "Value" "LED_RGAB"
-			(at 0 4.4 0)
-			(layer "F.Fab")
-			(effects
-				(font
-					(size 1 1)
-					(thickness 0.15)
-				)
-			)
-		)
-		(property "Footprint" "lcsc:LED-ARRAY-SMD_4P-L2.0-W1.3-BR_HandSolder"
-			(at 0 0 0)
+			(at 0 4.4 180)
+			(layer "F.Fab")
+			(effects
+				(font
+					(size 1 1)
+					(thickness 0.15)
+				)
+			)
+		)
+		(property "Footprint" "discrete:LED_RGB_XL-2012RGBC_2.0x1.2mm_HandSolder"
+			(at 0 0 180)
 			(layer "F.Fab")
 			(hide yes)
@@
 		)
 		(property "Datasheet" "https://www.lcsc.com/datasheet/lcsc_datasheet_2211030000_XINGLIGHT-XL-2012RGBC_C965848.pdf"
-			(at 0 0 0)
+			(at 0 0 180)
 			(layer "F.Fab")
 			(hide yes)
@@
 		)
 		(property "Description" "RGB LED, red/green/anode/blue"
-			(at 0 0 0)
+			(at 0 0 180)
 			(layer "F.Fab")
 			(hide yes)
@@
 			)
 		)
-		(property ki_fp_filters "LED* LED_SMD:* LED_THT:*")
+		(property ki_fp_filters "LED*XL?2012RGBC*")
 		(sheetname "Root")
-		(sheetfile "led-jig-mini.kicad_sch")
+		(sheetfile "led-micro.kicad_sch")
 		(attr smd)
+		(fp_line
+			(start 1.6 0.1)
+			(end 1.6 -0.1)
+			(stroke
+				(width 0.12)
+				(type default)
+			)
+			(layer "F.SilkS")
+		)
+		(fp_line
+			(start 0.4 -0.75)
+			(end -0.4 -0.75)
+			(stroke
+				(width 0.12)
+				(type default)
+			)
+			(layer "F.SilkS")
+		)
 		(fp_line
 			(start 0.1 0)
@@
 				(width 0.2)
 				(type solid)
+			)
+			(layer "F.SilkS")
+		)
+		(fp_line
+			(start -0.4 0.75)
+			(end 0.4 0.75)
+			(stroke
+				(width 0.12)
+				(type default)
 			)
 			(layer "F.SilkS")
@@
 		)
 		(fp_rect
-			(start -1.565 -0.775)
-			(end 1.565 0.775)
+			(start -1.75 -0.9)
+			(end 1.75 0.9)
 			(stroke
 				(width 0.05)
@@
 			(layer "F.CrtYd")
 		)
-		(fp_circle
-			(center 1 0.63)
-			(end 1.03 0.63)
-			(stroke
-				(width 0.06)
-				(type solid)
+		(fp_rect
+			(start -1 -0.65)
+			(end 1 0.65)
+			(stroke
+				(width 0.1)
+				(type default)
 			)
 			(fill none)
@@
 		)
 		(fp_text user "${REFERENCE}"
-			(at 0 0 0)
+			(at 0 0 180)
 			(layer "F.Fab")
 			(effects
@@
 		(property ki_fp_filters "R_*")
 		(sheetname "Root")
-		(sheetfile "led-jig-mini.kicad_sch")
+		(sheetfile "led-micro.kicad_sch")
 		(attr smd)
 		(fp_line
@@
 		(property ki_fp_filters "Connector*:*_1x??_*")
 		(sheetname "Root")
-		(sheetfile "led-jig-mini.kicad_sch")
+		(sheetfile "led-micro.kicad_sch")
 		(attr through_hole)
 		(fp_line
@@
 		(property ki_fp_filters "Connector*:*_1x??_*")
 		(sheetname "Root")
-		(sheetfile "led-jig-mini.kicad_sch")
+		(sheetfile "led-micro.kicad_sch")
 		(attr through_hole)
 		(fp_line
@@
 		(property ki_fp_filters "R_*")
 		(sheetname "Root")
-		(sheetfile "led-jig-mini.kicad_sch")
+		(sheetfile "led-micro.kicad_sch")
 		(attr smd)
 		(fp_line
@@
 		(property ki_fp_filters "R_*")
 		(sheetname "Root")
-		(sheetfile "led-jig-mini.kicad_sch")
+		(sheetfile "led-micro.kicad_sch")
 		(attr smd)
 		(fp_line
@@
 		(property ki_fp_filters "R_*")
 		(sheetname "Root")
-		(sheetfile "led-jig-mini.kicad_sch")
+		(sheetfile "led-micro.kicad_sch")
 		(attr smd)
 		(fp_line

Commit message: Update URL to pcb.smkent.net on remaining boards
Other:
- board text added: "pcb.smkent.net"
- board text removed: "github.com/smkent/pcb"
Changed lines of the file:
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@@
 		(layer "Edge.Cuts")
 	)
-	(gr_text "github.com/smkent/pcb"
+	(gr_text "pcb.smkent.net"
 		(at 128.778 100.33 270)
 		(layer "B.SilkS")
