File: pcb/stackable2/esp-lcd-dev/esp-lcd-dev.kicad_sch (KiCad schematic)
At the start: 29 parts, among them J1 JST XH/PH, J2 Qwiic, J3 Qwiic, J4 STEMMA-Signal, J5 JST SH, J6 Pin headers, J7 Pin headers, J8 Pin headers, Q1 2N7002DW, U1 VEML7700

Commit message: Rename `connectors` symbol and footprint libraries to `connector`
Parts:
- J2, J3: footprint connectors:Qwiic-SMD-horizontal-logo-bottom-pinout -> connector:Qwiic-SMD-horizontal-logo-bottom-pinout; symbol connectors:Qwiic -> connector:Qwiic
- J4: footprint connectors:STEMMA-Signal-SMD-horizontal -> connector:STEMMA-Signal-SMD-horizontal; symbol connectors:STEMMA-Signal -> connector:STEMMA-Signal
- J5: footprint connectors:JST_SH_SM08B-SRSS-TB_1x08-1MP_P1.00mm_Horizontal -> connector:JST_SH_SM08B-SRSS-TB_1x08-1MP_P1.00mm_Horizontal
Changed lines of the file:
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@@
 	)
 	(symbol
-		(lib_id "connectors:Qwiic")
+		(lib_id "connector:Qwiic")
 		(at 58.42 132.08 0)
 		(unit 1)
@@
 			)
 		)
-		(property "Footprint" "connectors:Qwiic-SMD-horizontal-logo-bottom-pinout"
+		(property "Footprint" "connector:Qwiic-SMD-horizontal-logo-bottom-pinout"
 			(at 58.42 132.08 0)
 			(effects
@@
 	)
 	(symbol
-		(lib_id "connectors:STEMMA-Signal")
+		(lib_id "connector:STEMMA-Signal")
 		(at 110.49 132.08 0)
 		(unit 1)
@@
 			)
 		)
-		(property "Footprint" "connectors:STEMMA-Signal-SMD-horizontal"
+		(property "Footprint" "connector:STEMMA-Signal-SMD-horizontal"
 			(at 110.49 132.08 0)
 			(effects
@@
 			)
 		)
-		(property "Footprint" "connectors:JST_SH_SM08B-SRSS-TB_1x08-1MP_P1.00mm_Horizontal"
+		(property "Footprint" "connector:JST_SH_SM08B-SRSS-TB_1x08-1MP_P1.00mm_Horizontal"
 			(at 105.41 83.82 0)
 			(effects
@@
 	)
 	(symbol
-		(lib_id "connectors:Qwiic")
+		(lib_id "connector:Qwiic")
 		(at 77.47 132.08 0)
 		(unit 1)
@@
 			)
 		)
-		(property "Footprint" "connectors:Qwiic-SMD-horizontal-logo-bottom-pinout"
+		(property "Footprint" "connector:Qwiic-SMD-horizontal-logo-bottom-pinout"
 			(at 77.47 132.08 0)
 			(effects

Commit message: Rename `modules` symbol and footprint libraries to `module`
Parts:
- SM1: footprint modules:ESP32-C3-Super-Mini-Castellated-SMD-only -> module:ESP32-C3-Super-Mini-Castellated-SMD-only; symbol modules:ESP32-C3-Super-Mini -> module:ESP32-C3-Super-Mini
Changed lines of the file:
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@@
 	)
 	(symbol
-		(lib_id "modules:ESP32-C3-Super-Mini")
+		(lib_id "module:ESP32-C3-Super-Mini")
 		(at 53.34 39.37 0)
 		(unit 1)
@@
 			)
 		)
-		(property "Footprint" "modules:ESP32-C3-Super-Mini-Castellated-SMD-only"
+		(property "Footprint" "module:ESP32-C3-Super-Mini-Castellated-SMD-only"
 			(at 53.34 23.622 0)
 			(effects

Commit message: Migrate `2N7002DW` symbol from `lcsc` to `discrete`
Parts:
- Q1: symbol lcsc:2N7002DW -> discrete:2N7002DW
Changed lines of the file:
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@@
 	)
 	(symbol
-		(lib_id "lcsc:2N7002DW")
+		(lib_id "discrete:2N7002DW")
 		(at 223.52 54.61 270)
 		(unit 2)
@@
 	)
 	(symbol
-		(lib_id "lcsc:2N7002DW")
+		(lib_id "discrete:2N7002DW")
 		(at 223.52 34.29 270)
 		(unit 1)

Commit message: Migrate `VEML6030`, `VEML7700` symbols from `lcsc` to `discrete`
Parts:
- U1: symbol lcsc:VEML7700 -> discrete:VEML7700
Changed lines of the file:
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@@
 	)
 	(symbol
-		(lib_id "lcsc:VEML7700")
+		(lib_id "discrete:VEML7700")
 		(at 111.76 38.1 0)
 		(unit 1)

Commit message: Recreate WS2812B-2020 footprints in `discrete` footprint library
Parts:
- LED2, LED3, LED4, LED5, LED6, LED7: footprint lcsc:LED-SMD_4P-L2.0-W2.0-BR-1 -> discrete:LED_WS2812B-2020_PLCC4_2.0x2.0mm_HandSolder
Changed lines of the file:
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@@
 			)
 		)
-		(property "Footprint" "lcsc:LED-SMD_4P-L2.0-W2.0-BR-1"
+		(property "Footprint" "discrete:LED_WS2812B-2020_PLCC4_2.0x2.0mm_HandSolder"
 			(at 207.01 147.32 0)
 			(effects
@@
 			)
 		)
-		(property "Footprint" "lcsc:LED-SMD_4P-L2.0-W2.0-BR-1"
+		(property "Footprint" "discrete:LED_WS2812B-2020_PLCC4_2.0x2.0mm_HandSolder"
 			(at 247.65 147.32 0)
 			(effects
@@
 			)
 		)
-		(property "Footprint" "lcsc:LED-SMD_4P-L2.0-W2.0-BR-1"
+		(property "Footprint" "discrete:LED_WS2812B-2020_PLCC4_2.0x2.0mm_HandSolder"
 			(at 267.97 147.32 0)
 			(effects
@@
 			)
 		)
-		(property "Footprint" "lcsc:LED-SMD_4P-L2.0-W2.0-BR-1"
+		(property "Footprint" "discrete:LED_WS2812B-2020_PLCC4_2.0x2.0mm_HandSolder"
 			(at 227.33 147.32 0)
 			(effects
@@
 			)
 		)
-		(property "Footprint" "lcsc:LED-SMD_4P-L2.0-W2.0-BR-1"
+		(property "Footprint" "discrete:LED_WS2812B-2020_PLCC4_2.0x2.0mm_HandSolder"
 			(at 186.69 147.32 0)
 			(effects
@@
 			)
 		)
-		(property "Footprint" "lcsc:LED-SMD_4P-L2.0-W2.0-BR-1"
+		(property "Footprint" "discrete:LED_WS2812B-2020_PLCC4_2.0x2.0mm_HandSolder"
 			(at 166.37 147.32 0)
 			(effects

Commit message: Migrate VEML6030, VEML7700 footprints from `lcsc` to `discrete`
Parts:
- U1: footprint lcsc:SENSORS-SMD_VEML7700-TR -> discrete:Sensor_VEML7700-TR; LCSC Part (none) -> C504893
Changed lines of the file:
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@@
 			)
 		)
-		(property "Footprint" "lcsc:SENSORS-SMD_VEML7700-TR"
+		(property "Footprint" "discrete:Sensor_VEML7700-TR"
 			(at 114.3 55.88 0)
 			(effects
@@
 			(at 111.76 38.1 0)
 			(effects
+				(font
+					(size 1.27 1.27)
+				)
+				(hide yes)
+			)
+		)
+		(property "LCSC Part" "C504893"
+			(at 111.76 38.1 0)
+			(effects

Commit message: Migrate 0603 capacitor hand soldering footprint to `discrete`
Parts:
- C2, C3, C6, C7: footprint custom:C_0603_1608Metric_Pad1.08x0.95mm_HandSolder -> discrete:C_0603_1608Metric_Pad1.08x0.95mm_HandSolder
Changed lines of the file:
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@@
 			)
 		)
-		(property "Footprint" "custom:C_0603_1608Metric_Pad1.08x0.95mm_HandSolder"
+		(property "Footprint" "discrete:C_0603_1608Metric_Pad1.08x0.95mm_HandSolder"
 			(at 135.89 120.65 0)
 			(effects
@@
 			)
 		)
-		(property "Footprint" "custom:C_0603_1608Metric_Pad1.08x0.95mm_HandSolder"
+		(property "Footprint" "discrete:C_0603_1608Metric_Pad1.08x0.95mm_HandSolder"
 			(at 156.21 58.42 0)
 			(effects
@@
 			)
 		)
-		(property "Footprint" "custom:C_0603_1608Metric_Pad1.08x0.95mm_HandSolder"
+		(property "Footprint" "discrete:C_0603_1608Metric_Pad1.08x0.95mm_HandSolder"
 			(at 146.05 120.65 0)
 			(effects
@@
 			)
 		)
-		(property "Footprint" "custom:C_0603_1608Metric_Pad1.08x0.95mm_HandSolder"
+		(property "Footprint" "discrete:C_0603_1608Metric_Pad1.08x0.95mm_HandSolder"
 			(at 167.64 34.29 0)
 			(effects
