File: pcb/stackable2/esp-rgb-driver/esp-rgb-driver.kicad_sch (KiCad schematic)
At the start: 45 parts, among them J0 Barrel Jack, J1 JST PH, J2 JST PH, J3 JST PH, J4 JST PH, J5 STEMMA-Signal, J6 STEMMA-Signal, J7 JST SH, J8 Qwiic, Q1 ZC010DNG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

Commit message: Migrate `TPS54202DDCR` symbol from `lcsc` to `ic`
Parts:
- U1: symbol lcsc:TPS54202DDCR -> ic:TPS54202DDCR
Changed lines of the file:
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@@
 	(symbol
 		(lib_name "TPS54202DDCR_1")
-		(lib_id "lcsc:TPS54202DDCR")
+		(lib_id "ic:TPS54202DDCR")
 		(at 59.69 78.74 0)
 		(unit 1)

Commit message: Migrate `WS2811F` symbol from `lcsc` to `ic`
Parts:
- U3, U4, U5, U6: symbol lcsc:WS2811F -> ic:WS2811F
Changed lines of the file:
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@@
 	)
 	(symbol
-		(lib_id "lcsc:WS2811F")
+		(lib_id "ic:WS2811F")
 		(at 147.32 64.77 0)
 		(unit 1)
@@
 	)
 	(symbol
-		(lib_id "lcsc:WS2811F")
+		(lib_id "ic:WS2811F")
 		(at 147.32 34.29 0)
 		(unit 1)
@@
 	)
 	(symbol
-		(lib_id "lcsc:WS2811F")
+		(lib_id "ic:WS2811F")
 		(at 147.32 111.76 0)
 		(unit 1)
@@
 	)
 	(symbol
-		(lib_id "lcsc:WS2811F")
+		(lib_id "ic:WS2811F")
 		(at 147.32 139.7 0)
 		(unit 1)

Commit message: Update esp-3dp and esp-rgb-driver to use new `SN74LVC1T45Z6` symbol
Parts:
- U2: value SN74LVC1T45DRL -> SN74LVC1T45Z6; symbol Logic_LevelTranslator:SN74LVC1T45DRL -> ic:SN74LVC1T45Z6; LCSC Part (none) -> C441819
Changed lines of the file:
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@@
 	)
 	(symbol
-		(lib_id "Logic_LevelTranslator:SN74LVC1T45DRL")
+		(lib_id "ic:SN74LVC1T45Z6")
 		(at 50.8 124.46 0)
 		(unit 1)
@@
 			)
 		)
-		(property "Value" "SN74LVC1T45DRL"
+		(property "Value" "SN74LVC1T45Z6"
 			(at 68.58 120.6814 0)
 			(effects
@@
 			)
 		)
-		(property "Datasheet" "http://www.ti.com/lit/ds/symlink/sn74lvc1t45.pdf"
+		(property "Datasheet" "https://www.diodes.com/assets/Datasheets/74LVC1T45.pdf"
 			(at 27.94 140.97 0)
 			(effects
@@
 			(at 50.8 124.46 0)
 			(effects
+				(font
+					(size 1.27 1.27)
+				)
+				(hide yes)
+			)
+		)
+		(property "LCSC Part" "C441819"
+			(at 50.8 124.46 0)
+			(effects

Commit message: Update esp-rgb-driver to use new `NC7WZ14P6X` symbol
Parts:
- U10, U11, U12, U7, U8, U9: value NC7WZ14 -> NC7WZ14P6X; symbol 74xGxx:Inverter_Schmitt_Dual -> ic:NC7WZ14P6X; LCSC Part (none) -> C5207816
Changed lines of the file:
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@@
 	)
 	(symbol
-		(lib_id "74xGxx:Inverter_Schmitt_Dual")
+		(lib_id "ic:NC7WZ14P6X")
 		(at 181.61 48.26 0)
 		(unit 1)
@@
 			)
 		)
-		(property "Value" "NC7WZ14"
+		(property "Value" "NC7WZ14P6X"
 			(at 183.8041 38.1 0)
 			(effects
@@
 			)
 		)
-		(property "Description" "Dual schmitt inverter"
+		(property "Description" "Dual schmitt inverter, VCC from 1.65 to 5.5 V, SOT-363-6"
+			(at 181.61 48.26 0)
+			(effects
+				(font
+					(size 1.27 1.27)
+				)
+				(hide yes)
+			)
+		)
+		(property "LCSC Part" "C5207816"
 			(at 181.61 48.26 0)
 			(effects
@@
 	)
 	(symbol
-		(lib_id "74xGxx:Inverter_Schmitt_Dual")
+		(lib_id "ic:NC7WZ14P6X")
 		(at 245.11 128.27 0)
 		(unit 1)
@@
 			)
 		)
-		(property "Value" "NC7WZ14"
+		(property "Value" "NC7WZ14P6X"
 			(at 247.3041 118.11 0)
 			(effects
@@
 			)
 		)
-		(property "Description" "Dual schmitt inverter"
+		(property "Description" "Dual schmitt inverter, VCC from 1.65 to 5.5 V, SOT-363-6"
+			(at 245.11 128.27 0)
+			(effects
+				(font
+					(size 1.27 1.27)
+				)
+				(hide yes)
+			)
+		)
+		(property "LCSC Part" "C5207816"
 			(at 245.11 128.27 0)
 			(effects
@@
 	)
 	(symbol
-		(lib_id "74xGxx:Inverter_Schmitt_Dual")
+		(lib_id "ic:NC7WZ14P6X")
 		(at 245.11 86.36 0)
 		(unit 1)
@@
 			)
 		)
-		(property "Value" "NC7WZ14"
+		(property "Value" "NC7WZ14P6X"
 			(at 247.3041 76.2 0)
 			(effects
@@
 			)
 		)
-		(property "Description" "Dual schmitt inverter"
+		(property "Description" "Dual schmitt inverter, VCC from 1.65 to 5.5 V, SOT-363-6"
+			(at 245.11 86.36 0)
+			(effects
+				(font
+					(size 1.27 1.27)
+				)
+				(hide yes)
+			)
+		)
+		(property "LCSC Part" "C5207816"
 			(at 245.11 86.36 0)
 			(effects
@@
 	)
 	(symbol
-		(lib_id "74xGxx:Inverter_Schmitt_Dual")
+		(lib_id "ic:NC7WZ14P6X")
 		(at 245.11 48.26 0)
 		(unit 1)
@@
 			)
 		)
-		(property "Value" "NC7WZ14"
+		(property "Value" "NC7WZ14P6X"
 			(at 247.3041 38.1 0)
 			(effects
@@
 			)
 		)
-		(property "Description" "Dual schmitt inverter"
+		(property "Description" "Dual schmitt inverter, VCC from 1.65 to 5.5 V, SOT-363-6"
+			(at 245.11 48.26 0)
+			(effects
+				(font
+					(size 1.27 1.27)
+				)
+				(hide yes)
+			)
+		)
+		(property "LCSC Part" "C5207816"
 			(at 245.11 48.26 0)
 			(effects
@@
 	)
 	(symbol
-		(lib_id "74xGxx:Inverter_Schmitt_Dual")
+		(lib_id "ic:NC7WZ14P6X")
 		(at 181.61 86.36 0)
 		(unit 1)
@@
 			)
 		)
-		(property "Value" "NC7WZ14"
+		(property "Value" "NC7WZ14P6X"
 			(at 183.8041 76.2 0)
 			(effects
@@
 			)
 		)
-		(property "Description" "Dual schmitt inverter"
+		(property "Description" "Dual schmitt inverter, VCC from 1.65 to 5.5 V, SOT-363-6"
+			(at 181.61 86.36 0)
+			(effects
+				(font
+					(size 1.27 1.27)
+				)
+				(hide yes)
+			)
+		)
+		(property "LCSC Part" "C5207816"
 			(at 181.61 86.36 0)
 			(effects
@@
 	)
 	(symbol
-		(lib_id "74xGxx:Inverter_Schmitt_Dual")
+		(lib_id "ic:NC7WZ14P6X")
 		(at 181.61 128.27 0)
 		(unit 1)
@@
 			)
 		)
-		(property "Value" "NC7WZ14"
+		(property "Value" "NC7WZ14P6X"
 			(at 183.8041 118.11 0)
 			(effects
@@
 			)
 		)
-		(property "Description" "Dual schmitt inverter"
+		(property "Description" "Dual schmitt inverter, VCC from 1.65 to 5.5 V, SOT-363-6"
+			(at 181.61 128.27 0)
+			(effects
+				(font
+					(size 1.27 1.27)
+				)
+				(hide yes)
+			)
+		)
+		(property "LCSC Part" "C5207816"
 			(at 181.61 128.27 0)
 			(effects

Commit message: Migrate `LED_0402_1005Metric` from `led` to `discrete`
Parts:
- LED1: footprint led:LED_0402_1005Metric -> discrete:LED_0402_1005Metric
Changed lines of the file:
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@@
 			)
 		)
-		(property "Footprint" "led:LED_0402_1005Metric"
+		(property "Footprint" "discrete:LED_0402_1005Metric"
 			(at 114.3 57.15 0)
 			(effects

Commit message: Migrate esp-rgb-driver to new DC-050 DC jack footprint
Parts:
- J0: footprint custom:DC-IN_DC-050-2.0-BB_rev2 -> connector:BarrelJack_DC-050_SMT_Horizontal
Changed lines of the file:
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@@
 			)
 		)
-		(property "Footprint" "custom:DC-IN_DC-050-2.0-BB_rev2"
+		(property "Footprint" "connector:BarrelJack_DC-050_SMT_Horizontal"
 			(at 86.36 31.496 0)
 			(effects

Commit message: Migrate 0805 capacitor hand soldering footprint to `discrete`
Parts:
- C5, C6, C7: footprint custom:C_0805_2012Metric_Pad1.18x1.45mm_HandSolder -> discrete:C_0805_2012Metric_Pad1.18x1.45mm_HandSolder
Changed lines of the file:
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@@
 			)
 		)
-		(property "Footprint" "custom:C_0805_2012Metric_Pad1.18x1.45mm_HandSolder"
+		(property "Footprint" "discrete:C_0805_2012Metric_Pad1.18x1.45mm_HandSolder"
 			(at 91.44 83.82 0)
 			(effects
@@
 			)
 		)
-		(property "Footprint" "custom:C_0805_2012Metric_Pad1.18x1.45mm_HandSolder"
+		(property "Footprint" "discrete:C_0805_2012Metric_Pad1.18x1.45mm_HandSolder"
 			(at 100.33 83.82 0)
 			(effects
@@
 			)
 		)
-		(property "Footprint" "custom:C_0805_2012Metric_Pad1.18x1.45mm_HandSolder"
+		(property "Footprint" "discrete:C_0805_2012Metric_Pad1.18x1.45mm_HandSolder"
 			(at 109.22 83.82 0)
 			(effects

Commit message: Migrate 0603 capacitor hand soldering footprint to `discrete`
Parts:
- C1, C2: footprint custom:C_0603_1608Metric_Pad1.08x0.95mm_HandSolder -> discrete:C_0603_1608Metric_Pad1.08x0.95mm_HandSolder
Changed lines of the file:
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@@
 			)
 		)
-		(property "Footprint" "custom:C_0603_1608Metric_Pad1.08x0.95mm_HandSolder"
+		(property "Footprint" "discrete:C_0603_1608Metric_Pad1.08x0.95mm_HandSolder"
 			(at 24.13 81.28 0)
 			(effects
@@
 			)
 		)
-		(property "Footprint" "custom:C_0603_1608Metric_Pad1.08x0.95mm_HandSolder"
+		(property "Footprint" "discrete:C_0603_1608Metric_Pad1.08x0.95mm_HandSolder"
 			(at 33.02 81.28 0)
 			(effects
