File: pcb/jigs/neopixel-micro/neopixel-micro.kicad_pcb (KiCad board)
At the start: 2 copper layers, 13 x 13 mm, 20 parts, among them J1 Conn_01x02, J2 Conn_01x02, J3 Conn_01x01, J4 Conn_01x01

Commit message: Migrate 0603 capacitor hand soldering footprint to `discrete`
Parts:
- C1, C2: footprint custom:C_0603_1608Metric_Pad1.08x0.95mm_HandSolder -> discrete:C_0603_1608Metric_Pad1.08x0.95mm_HandSolder
Changed lines of the file:
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@@
 		)
 	)
-	(footprint "custom:C_0603_1608Metric_Pad1.08x0.95mm_HandSolder"
+	(footprint "discrete:C_0603_1608Metric_Pad1.08x0.95mm_HandSolder"
 		(layer "F.Cu")
 		(at 130.155 102.87 180)
@@
 			)
 		)
-		(property "Footprint" "custom:C_0603_1608Metric_Pad1.08x0.95mm_HandSolder"
+		(property "Footprint" "discrete:C_0603_1608Metric_Pad1.08x0.95mm_HandSolder"
 			(at 0 0 180)
 			(unlocked yes)
@@
 		)
 	)
-	(footprint "custom:C_0603_1608Metric_Pad1.08x0.95mm_HandSolder"
+	(footprint "discrete:C_0603_1608Metric_Pad1.08x0.95mm_HandSolder"
 		(layer "B.Cu")
 		(at 130.155 102.87 180)
@@
 			)
 		)
-		(property "Footprint" "custom:C_0603_1608Metric_Pad1.08x0.95mm_HandSolder"
+		(property "Footprint" "discrete:C_0603_1608Metric_Pad1.08x0.95mm_HandSolder"
 			(at 0 0 0)
 			(unlocked yes)

Commit message: Migrate neopixel-micro to regular courtyard size WS2812 footprint
Parts:
- D1, D2: footprint custom:LED_WS2812B_PLCC4_5.0x5.0mm_P3.2mm_simple_small_courtyard -> custom:LED_WS2812B_PLCC4_5.0x5.0mm_P3.2mm_simple
Changed lines of the file:
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@@
 		)
 	)
-	(footprint "custom:LED_WS2812B_PLCC4_5.0x5.0mm_P3.2mm_simple_small_courtyard"
+	(footprint "custom:LED_WS2812B_PLCC4_5.0x5.0mm_P3.2mm_simple"
 		(layer "B.Cu")
 		(at 134.405 97.84 90)
@@
 			)
 		)
-		(property "Footprint" "custom:LED_WS2812B_PLCC4_5.0x5.0mm_P3.2mm_simple_small_courtyard"
+		(property "Footprint" "custom:LED_WS2812B_PLCC4_5.0x5.0mm_P3.2mm_simple"
 			(at 0 0 -90)
 			(unlocked yes)
@@
 			(layer "B.SilkS")
 		)
-		(fp_rect
-			(start -3.2 2.5)
-			(end 3.2 -2.5)
-			(stroke
-				(width 0.05)
-				(type default)
-			)
-			(fill none)
+		(fp_line
+			(start 3.45 -2.75)
+			(end -3.45 -2.75)
+			(stroke
+				(width 0.05)
+				(type solid)
+			)
+			(layer "B.CrtYd")
+		)
+		(fp_line
+			(start -3.45 -2.75)
+			(end -3.45 2.75)
+			(stroke
+				(width 0.05)
+				(type solid)
+			)
+			(layer "B.CrtYd")
+		)
+		(fp_line
+			(start 3.45 2.75)
+			(end 3.45 -2.75)
+			(stroke
+				(width 0.05)
+				(type solid)
+			)
+			(layer "B.CrtYd")
+		)
+		(fp_line
+			(start -3.45 2.75)
+			(end 3.45 2.75)
+			(stroke
+				(width 0.05)
+				(type solid)
+			)
 			(layer "B.CrtYd")
 		)
@@
 		)
 	)
-	(footprint "custom:LED_WS2812B_PLCC4_5.0x5.0mm_P3.2mm_simple_small_courtyard"
+	(footprint "custom:LED_WS2812B_PLCC4_5.0x5.0mm_P3.2mm_simple"
 		(layer "B.Cu")
 		(at 128.405 97.84 90)
@@
 			)
 		)
-		(property "Footprint" "custom:LED_WS2812B_PLCC4_5.0x5.0mm_P3.2mm_simple_small_courtyard"
+		(property "Footprint" "custom:LED_WS2812B_PLCC4_5.0x5.0mm_P3.2mm_simple"
 			(at 0 0 -90)
 			(unlocked yes)
@@
 			(layer "B.SilkS")
 		)
-		(fp_rect
-			(start -3.2 2.5)
-			(end 3.2 -2.5)
-			(stroke
-				(width 0.05)
-				(type default)
-			)
-			(fill none)
-			(layer "B.CrtYd")
-		)
+		(fp_line
+			(start 3.45 -2.75)
+			(end -3.45 -2.75)
+			(stroke
+				(width 0.05)
+				(type solid)
+			)
+			(layer "B.CrtYd")
+		)
+		(fp_line
+			(start -3.45 -2.75)
+			(end -3.45 2.75)
+			(stroke
+				(width 0.05)
+				(type solid)
+			)
+			(layer "B.CrtYd")
+		)
+		(fp_line
+			(start 3.45 2.75)
+			(end 3.45 -2.75)
+			(stroke
+				(width 0.05)
+				(type solid)
+			)
+			(layer "B.CrtYd")
+		)
+		(fp_line
+			(start -3.45 2.75)
+			(end 3.45 2.75)
+			(stroke
+				(width 0.05)
+				(type solid)
+			)
+			(layer "B.CrtYd")
+		)

Commit message: Migrate `LED_WS2812B_PLCC4_5.0x5.0mm_P3.2mm` footprint to `discrete`
Parts:
- D1, D2: footprint custom:LED_WS2812B_PLCC4_5.0x5.0mm_P3.2mm_simple -> discrete:LED_WS2812B_PLCC4_5.0x5.0mm_P3.2mm
Changed lines of the file:
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@@
 		)
 	)
-	(footprint "custom:LED_WS2812B_PLCC4_5.0x5.0mm_P3.2mm_simple"
+	(footprint "discrete:LED_WS2812B_PLCC4_5.0x5.0mm_P3.2mm"
 		(layer "B.Cu")
 		(at 134.405 97.84 90)
@@
 			)
 		)
-		(property "Footprint" "custom:LED_WS2812B_PLCC4_5.0x5.0mm_P3.2mm_simple"
+		(property "Footprint" "discrete:LED_WS2812B_PLCC4_5.0x5.0mm_P3.2mm"
 			(at 0 0 -90)
 			(unlocked yes)
@@
 		)
 	)
-	(footprint "custom:LED_WS2812B_PLCC4_5.0x5.0mm_P3.2mm_simple"
+	(footprint "discrete:LED_WS2812B_PLCC4_5.0x5.0mm_P3.2mm"
 		(layer "B.Cu")
 		(at 128.405 97.84 90)
@@
 			)
 		)
-		(property "Footprint" "custom:LED_WS2812B_PLCC4_5.0x5.0mm_P3.2mm_simple"
-			(at 0 0 -90)
-			(unlocked yes)
+		(property "Footprint" "discrete:LED_WS2812B_PLCC4_5.0x5.0mm_P3.2mm"
+			(at 0 0 -90)
+			(unlocked yes)
