File: pcb/jigs/breadboard-power/breadboard-power.kicad_pcb (KiCad board)
At the start: 2 copper layers, 51.3 x 22 mm, 30 parts, among them J0 USB_C_Receptacle_PowerOnly_6P, J1 Barrel_Jack_Switch, J2 Barrel_Jack_Switch, J4 USB_C_Receptacle_PowerOnly_6P, Q1 AO3401A, Q2 AO3401A, Q3 AO3401A, Q4 AO3401A, SW1 SW_SPDT, SW2 SW_SPDT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

Commit message: Migrate `SW-SMD_3P-P1.50_L2.7-W6.6` footprint to `electromechanical`
Parts:
- SW3: footprint lcsc:SW-SMD_3P-P1.50_L2.7-W6.6 -> electromechanical:SW-SMD_3P-P1.50_L2.7-W6.6
Changed lines of the file:
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@@
 		)
 	)
-	(footprint "lcsc:SW-SMD_3P-P1.50_L2.7-W6.6"
+	(footprint "electromechanical:SW-SMD_3P-P1.50_L2.7-W6.6"
 		(layer "F.Cu")
 		(at 204.47 92.42)
@@
 			)
 		)
-		(property "Footprint" "lcsc:SW-SMD_3P-P1.50_L2.7-W6.6"
+		(property "Footprint" "electromechanical:SW-SMD_3P-P1.50_L2.7-W6.6"
 			(at 0 0 0)
 			(layer "F.Fab")

Commit message: Migrate breadboard-power to use `SW_SPDT_PCM12` footprint
Parts:
- SW3: footprint electromechanical:SW-SMD_3P-P1.50_L2.7-W6.6 -> electromechanical:SW_SPDT_PCM12
- moved SW3 0.12 mm to (204.5, 92.5)

Commit message: Recreate 3-pin SPDT THT slide switch footprint to replace LCSC footprint
Parts:
- SW1, SW2: footprint custom:SW-TH_DEALON_SS-12D01-GX_simple -> electromechanical:SW_Slide-03_SPDT_P2.50mm_THT

Commit message: Migrate custom USB-C 6P receptacle footprint to `connector`
Parts:
- J0, J4: footprint custom:USB_C_Receptacle_GCT_USB4125-xx-x_6P_TopMnt_Horizontal_handsolder -> connector:USB_C_Receptacle_GCT_USB4125-xx-x_6P_TopMnt_Horizontal_HandSolder
Changed lines of the file:
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@@
 		)
 	)
-	(footprint "custom:USB_C_Receptacle_GCT_USB4125-xx-x_6P_TopMnt_Horizontal_handsolder"
+	(footprint "connector:USB_C_Receptacle_GCT_USB4125-xx-x_6P_TopMnt_Horizontal_HandSolder"
 		(layer "F.Cu")
 		(at 224.536 79.502 180)
@@
 			)
 		)
-		(property "Footprint" "custom:USB_C_Receptacle_GCT_USB4125-xx-x_6P_TopMnt_Horizontal_handsolder"
+		(property "Footprint" "connector:USB_C_Receptacle_GCT_USB4125-xx-x_6P_TopMnt_Horizontal_HandSolder"
 			(at 0 0 180)
 			(unlocked yes)
@@
 		)
 	)
-	(footprint "custom:USB_C_Receptacle_GCT_USB4125-xx-x_6P_TopMnt_Horizontal_handsolder"
+	(footprint "connector:USB_C_Receptacle_GCT_USB4125-xx-x_6P_TopMnt_Horizontal_HandSolder"
 		(layer "F.Cu")
 		(at 184.152 79.502 180)
@@
 			)
 		)
-		(property "Footprint" "custom:USB_C_Receptacle_GCT_USB4125-xx-x_6P_TopMnt_Horizontal_handsolder"
+		(property "Footprint" "connector:USB_C_Receptacle_GCT_USB4125-xx-x_6P_TopMnt_Horizontal_HandSolder"
 			(at 0 0 180)
 			(unlocked yes)

Commit message: Migrate `D_SOD-323_HandSoldering` footprint to `package`
Parts:
- D1, D2: footprint custom:D_SOD-323_HandSoldering_simple -> package:D_SOD-323_HandSoldering
Changed lines of the file:
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@@
 		)
 	)
-	(footprint "custom:D_SOD-323_HandSoldering_simple"
+	(footprint "package:D_SOD-323_HandSoldering"
 		(layer "B.Cu")
 		(at 201.549 92.583 90)
@@
 		(tags "SOD-323")
 		(property "Reference" "D1"
-			(at 0 1.85 90)
+			(at 0 1.85 -90)
 			(layer "B.SilkS")
 			(hide yes)
@@
 		)
 		(property "Value" "1N4148WS"
-			(at 0.1 -1.9 90)
-			(layer "B.Fab")
-			(effects
-				(font
-					(size 1 1)
-					(thickness 0.15)
-				)
-				(justify mirror)
-			)
-		)
-		(property "Footprint" "custom:D_SOD-323_HandSoldering_simple"
+			(at 0.1 -1.9 -90)
+			(layer "B.Fab")
+			(effects
+				(font
+					(size 1 1)
+					(thickness 0.15)
+				)
+				(justify mirror)
+			)
+		)
+		(property "Footprint" "package:D_SOD-323_HandSoldering"
 			(at 0 0 -90)
 			(unlocked yes)
@@
 		)
 		(property "Sim.Device" "D"
-			(at 0 0 -90)
+			(at 0 0 90)
 			(unlocked yes)
 			(layer "B.Fab")
@@
 		)
 		(property "Sim.Pins" "1=K 2=A"
-			(at 0 0 -90)
+			(at 0 0 90)
 			(unlocked yes)
 			(layer "B.Fab")
@@
 		(sheetfile "breadboard-power.kicad_sch")
 		(attr smd)
+		(fp_line
+			(start -2 0.3)
+			(end -2 -0.3)
+			(stroke
+				(width 0.1)
+				(type default)
+			)
+			(layer "B.SilkS")
+		)
 		(fp_poly
 			(pts
@@
 		)
 		(fp_text user "${REFERENCE}"
-			(at 0 1.85 90)
+			(at 0 1.85 -90)
 			(layer "B.Fab")
 			(effects
@@
 		)
 	)
-	(footprint "custom:D_SOD-323_HandSoldering_simple"
+	(footprint "package:D_SOD-323_HandSoldering"
 		(layer "B.Cu")
 		(at 207.3656 92.583 90)
@@
 		(tags "SOD-323")
 		(property "Reference" "D2"
-			(at 0 1.85 90)
+			(at 0 1.85 -90)
 			(layer "B.SilkS")
 			(hide yes)
@@
 		)
 		(property "Value" "1N4148WS"
-			(at 0.1 -1.9 90)
-			(layer "B.Fab")
-			(effects
-				(font
-					(size 1 1)
-					(thickness 0.15)
-				)
-				(justify mirror)
-			)
-		)
-		(property "Footprint" "custom:D_SOD-323_HandSoldering_simple"
+			(at 0.1 -1.9 -90)
+			(layer "B.Fab")
+			(effects
+				(font
+					(size 1 1)
+					(thickness 0.15)
+				)
+				(justify mirror)
+			)
+		)
+		(property "Footprint" "package:D_SOD-323_HandSoldering"
 			(at 0 0 -90)
 			(unlocked yes)
@@
 		)
 		(property "Sim.Device" "D"
-			(at 0 0 -90)
+			(at 0 0 90)
 			(unlocked yes)
 			(layer "B.Fab")
@@
 		)
 		(property "Sim.Pins" "1=K 2=A"
-			(at 0 0 -90)
+			(at 0 0 90)
 			(unlocked yes)
 			(layer "B.Fab")
@@
 		(sheetfile "breadboard-power.kicad_sch")
 		(attr smd)
+		(fp_line
+			(start -2 0.3)
+			(end -2 -0.3)
+			(stroke
+				(width 0.1)
+				(type default)
+			)
+			(layer "B.SilkS")
+		)
 		(fp_poly
 			(pts
@@
 		)
 		(fp_text user "${REFERENCE}"
-			(at 0 1.85 90)
-			(layer "B.Fab")
-			(effects
+			(at 0 1.85 -90)
+			(layer "B.Fab")
+			(effects

Commit message: Migrate 1206 fuse footprint to `discrete`, adjust pads, silkscreen
Parts:
- F1, F2: footprint custom:Fuse_1206_3216Metric_Pad1.42x1.75mm_HandSolder_simple -> discrete:Fuse_1206_3216Metric
