File: pcb/jigs/led-jig/led-jig.kicad_pcb (KiCad board)
At the start: 2 copper layers, 15.2 x 21.6 mm, 12 parts, among them J1 Conn_01x08, J2 Conn_01x08

Commit message: Update URL to pcb.smkent.net on remaining boards
Other:
- board text added: "LED Jig pcb.smkent.net 2024"
- board text removed: "JLCJLCJLCJLC"
- board text removed: "LED Jig smkent 2024"
Changed lines of the file:
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@@
 				(font
 					(size 1.27 1.27)
+					(thickness 0.15)
 				)
 			)
@@
 				(font
 					(size 1.27 1.27)
+					(thickness 0.15)
 				)
 			)
@@
 				(font
 					(size 1.27 1.27)
+					(thickness 0.15)
 				)
 			)
@@
 				(font
 					(size 1.27 1.27)
+					(thickness 0.15)
 				)
 			)
@@
 				(font
 					(size 1.27 1.27)
+					(thickness 0.15)
 				)
 			)
@@
 				(font
 					(size 1.27 1.27)
+					(thickness 0.15)
 				)
 			)
@@
 				(font
 					(size 1.27 1.27)
+					(thickness 0.15)
 				)
 			)
@@
 				(font
 					(size 1.27 1.27)
+					(thickness 0.15)
 				)
 			)
@@
 				(font
 					(size 1.27 1.27)
+					(thickness 0.15)
 				)
 			)
@@
 				(font
 					(size 1.27 1.27)
+					(thickness 0.15)
 				)
 			)
@@
 				(font
 					(size 1.27 1.27)
+					(thickness 0.15)
 				)
 			)
@@
 				(font
 					(size 1.27 1.27)
+					(thickness 0.15)
 				)
 			)
@@
 				(font
 					(size 1.27 1.27)
+					(thickness 0.15)
 				)
 			)
@@
 				(font
 					(size 1.27 1.27)
+					(thickness 0.15)
 				)
 			)
@@
 				(font
 					(size 1.27 1.27)
+					(thickness 0.15)
 				)
 			)
@@
 				(font
 					(size 1.27 1.27)
+					(thickness 0.15)
 				)
 			)
@@
 				(font
 					(size 1.27 1.27)
+					(thickness 0.15)
 				)
 			)
@@
 				(font
 					(size 1.27 1.27)
+					(thickness 0.15)
 				)
 			)
@@
 				(font
 					(size 1.27 1.27)
+					(thickness 0.15)
 				)
 			)
@@
 				(font
 					(size 1.27 1.27)
+					(thickness 0.15)
 				)
 			)
@@
 				(font
 					(size 1.27 1.27)
+					(thickness 0.15)
 				)
 			)
@@
 				(font
 					(size 1.27 1.27)
+					(thickness 0.15)
 				)
 			)
@@
 				(font
 					(size 1.27 1.27)
+					(thickness 0.15)
 				)
 			)
@@
 				(font
 					(size 1.27 1.27)
+					(thickness 0.15)
 				)
 			)
@@
 				(font
 					(size 1.27 1.27)
+					(thickness 0.15)
 				)
 			)
@@
 				(font
 					(size 1.27 1.27)
+					(thickness 0.15)
 				)
 			)
@@
 				(font
 					(size 1.27 1.27)
+					(thickness 0.15)
 				)
 			)
@@
 				(font
 					(size 1.27 1.27)
+					(thickness 0.15)
 				)
 			)
@@
 				(font
 					(size 1.27 1.27)
+					(thickness 0.15)
 				)
 			)
@@
 				(font
 					(size 1.27 1.27)
+					(thickness 0.15)
 				)
 			)
@@
 				(font
 					(size 1.27 1.27)
+					(thickness 0.15)
 				)
 				(justify mirror)
@@
 				(font
 					(size 1.27 1.27)
+					(thickness 0.15)
 				)
 				(justify mirror)
@@
 				(font
 					(size 1.27 1.27)
+					(thickness 0.15)
 				)
 				(justify mirror)
@@
 				(font
 					(size 1.27 1.27)
+					(thickness 0.15)
 				)
 				(justify mirror)
@@
 				(font
 					(size 1.27 1.27)
+					(thickness 0.15)
 				)
 				(justify mirror)
@@
 				(font
 					(size 1.27 1.27)
+					(thickness 0.15)
 				)
 				(justify mirror)
@@
 		(layer "Edge.Cuts")
 	)
-	(gr_text "JLCJLCJLCJLC"
-		(at 134.62 105.41 90)
+	(gr_text "LED Jig\npcb.smkent.net\n2024"
+		(at 132 105.41 90)
 		(layer "B.SilkS")
 		(effects
-			(font
-				(size 1 1)
-				(thickness 0.125)
-			)
-			(justify mirror)
-		)
-	)
-	(gr_text "LED Jig\nsmkent 2024"
-		(at 130.81 105.41 90)
-		(layer "B.SilkS")
-		(effects
