File: pcb/misc/esp-doorbell-dev/esp-doorbell-dev.kicad_pcb (KiCad board)
At the start: 2 copper layers, 28 x 97 mm, 29 parts, among them J1 JST XH, J2 Screw_Terminal_01x02, J3 JST XH/PH, J4 JST PH, Q1 BSS84, Q2 BSS84, Q3 BSS84, Q4 2N7002DW, Q5 BSS138, U1 WS2811F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

Commit message: Rework `HLK-LD2410C` to match KiCAD symbol conventions
Parts:
- SM4: value HLK-LD2410C-P -> HLK-LD2410C
Changed lines of the file:
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@@
 			)
 		)
-		(property "Value" "HLK-LD2410C-P"
+		(property "Value" "HLK-LD2410C"
 			(at 0 4 0)
 			(layer "F.Fab")
@@
 			)
 		)
-		(property "Datasheet" ""
+		(property "Datasheet" "https://www.lcsc.com/datasheet/lcsc_datasheet_2409141622_HI-LINK-HLK-LD2410C-P_C19723500.pdf"
 			(at 0 0 0)
 			(layer "F.Fab")
@@
 			)
 		)
-		(property "Description" ""
+		(property "Description" "Human Presence Sensor, Millimeter Wave Radar, Bluetooth Low Energy/UART module"
 			(at 0 0 0)
 			(layer "F.Fab")
@@
 			(net 25 "UART_1_RX")
 			(pinfunction "TXD")
-			(pintype "passive")
+			(pintype "output")
 		)
 		(pad "2" thru_hole circle
@@
 			(net 26 "UART_1_TX")
 			(pinfunction "RXD")
-			(pintype "passive")
+			(pintype "input")
 		)
 		(pad "3" thru_hole circle
@@
 			(net 42 "unconnected-(SM4-OUT-Pad3)")
 			(pinfunction "OUT")
-			(pintype "passive+no_connect")
+			(pintype "output+no_connect")
 		)
 		(pad "4" thru_hole circle

Commit message: Migrate HLK-LD2410C module footprint from `lcsc` to `module`
Parts:
- SM4: footprint lcsc:SENSOR-TH_HLK-LD2410C-P -> module:HLK-LD2410C-module
Changed lines of the file:
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@@
 		)
 	)
-	(footprint "lcsc:SENSOR-TH_HLK-LD2410C-P"
+	(footprint "module:HLK-LD2410C-module"
 		(layer "F.Cu")
 		(at 160 124.535)
@@
 			)
 		)
-		(property "Footprint" "lcsc:SENSOR-TH_HLK-LD2410C-P"
+		(property "Footprint" "module:HLK-LD2410C-module"
 			(at 0 0 0)
 			(layer "F.Fab")
@@
 			)
 		)
+		(property ki_fp_filters "*LD2410*")
 		(sheetname "Root")
 		(sheetfile "esp-doorbell-dev.kicad_sch")

Commit message: Migrate G3MB-202P footprint from `custom` to `discrete`
Parts:
- U2: footprint custom:RELAY-G3MB-202P-5VDC -> discrete:Relay_G3MB-202P
Changed lines of the file:
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@@
 		)
 	)
-	(footprint "custom:RELAY-G3MB-202P-5VDC"
+	(footprint "discrete:Relay_G3MB-202P"
 		(layer "F.Cu")
 		(at 160 72 180)
@@
 			)
 		)
-		(property "Footprint" "custom:RELAY-G3MB-202P-5VDC"
+		(property "Footprint" "discrete:Relay_G3MB-202P"
 			(at 0 0 0)
 			(layer "F.Fab")

Commit message: Migrate 3.5mm 1x02 terminal block footprint to `connector`
Parts:
- J2: footprint custom:TerminalBlock_Phoenix_PT-1,5-2-3.5-H_1x02_P3.50mm_Horizontal_custom -> connector:TerminalBlock_Phoenix_PT-1,5-2-3.5-H_1x02_P3.50mm_Horizontal
Changed lines of the file:
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@@
 		)
 	)
-	(footprint "custom:TerminalBlock_Phoenix_PT-1,5-2-3.5-H_1x02_P3.50mm_Horizontal_custom"
+	(footprint "connector:TerminalBlock_Phoenix_PT-1,5-2-3.5-H_1x02_P3.50mm_Horizontal"
 		(layer "F.Cu")
 		(at 168.75 65.2 180)
@@
 		(tags "THT Terminal Block Phoenix PT-1,5-2-3.5-H pitch 3.5mm size 7x7.6mm^2 drill 1.2mm pad 2.4mm")
 		(property "Reference" "J2"
-			(at 1.75 -4.16 0)
+			(at 1.75 -4.16 180)
 			(layer "F.SilkS")
 			(hide yes)
@@
 		)
 		(property "Value" "Screw_Terminal_01x02"
-			(at 1.75 5.56 0)
+			(at 1.75 5.56 180)
 			(layer "F.Fab")
 			(effects
@@
 			)
 		)
-		(property "Footprint" "custom:TerminalBlock_Phoenix_PT-1,5-2-3.5-H_1x02_P3.50mm_Horizontal_custom"
+		(property "Footprint" "connector:TerminalBlock_Phoenix_PT-1,5-2-3.5-H_1x02_P3.50mm_Horizontal"
 			(at 0 0 180)
 			(unlocked yes)
@@
 		)
 		(fp_text user "${REFERENCE}"
-			(at 1.75 2.4 0)
+			(at 1.75 2.4 180)
 			(layer "F.Fab")
 			(effects
@@
 		)
 		(group ""
-			(members "07a53385-ca07-4d88-b740-42a67fc1f4fd" "32cfda7d-fec0-49f2-819c-f8130cb32eb7"
-				"3e534e6e-5ec9-4dc9-914b-72e473619c3a" "69573439-3e49-486b-a7f3-2770c31c0cce"
-				"b3554183-ed61-4826-a97e-65d0001ee469"
+			(members "641187a2-7716-4708-a20e-96db075ead9c" "76e33859-fe86-4b57-aa84-eeaf48d6feeb"
+				"96e6ff36-92d7-4485-9754-175a3d444caf" "e76da3d8-2daa-46ba-a75b-85bbb8cbdd43"
+				"ef69a0a1-050a-475c-aad4-c686edf9d4a5"
 			)
 		)
 		(group ""
-			(members "920cfccc-919e-4e59-aae7-34d234171cf2" "a9398b63-27e1-47dd-880e-bf68111fc413"
-				"c731e760-7e48-4d20-9f58-dfc639147bf4" "ca41816d-24d7-47eb-bc98-62d6a4ab9e5b"
-				"d60053b4-1f17-43aa-bccb-05376575b74c"
-			)
-		)
+			(members "11622e4e-942a-4a50-9316-0c6f5bc8ac06" "22cc8786-69c5-4fe0-a606-a8937caecc0b"
+				"4e25c416-faee-472d-ba5e-83ad3df9886b" "59f8600a-11d3-41e2-aa97-2ce21684aba5"
+				"a6c140f7-a77d-4a5e-8e30-8f928970fb1c"
+			)
+		)

Commit message: Reduce custom footprint use on esp-doorbell-dev
Parts:
- Q4: footprint package:SOT-363_SC-70-6 -> package:SOT-363_SC-70-6_HandSolder
- Q5: footprint package:SOT-23 -> Package_TO_SOT_SMD:SOT-23
- R3, R4, R5: footprint custom:R_0603_1608Metric_Pad0.98x0.95mm_HandSolder_simple -> Resistor_SMD:R_0603_1608Metric_Pad0.98x0.95mm_HandSolder
Routing:
- net +3V3: track 18.7 -> 19.6 mm

Commit message: Migrate custom horizontal THT JST connector footprints to `connector`
Parts:
- J1: footprint custom:JST_XH_S6B-XH_1x06_P2.50mm_Horizontal -> connector:JST_XH_S6B-XH-2AW_1x06_P2.50mm_Horizontal
Changed lines of the file:
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@@
 		)
 	)
-	(footprint "custom:JST_XH_S6B-XH_1x06_P2.50mm_Horizontal"
+	(footprint "connector:JST_XH_S6B-XH-2AW_1x06_P2.50mm_Horizontal"
 		(layer "B.Cu")
 		(at 162.55 101.75 -90)
@@
 			)
 		)
-		(property "Footprint" "custom:JST_XH_S6B-XH_1x06_P2.50mm_Horizontal"
+		(property "Footprint" "connector:JST_XH_S6B-XH-2AW_1x06_P2.50mm_Horizontal"
 			(at 0 0 90)
 			(unlocked yes)

Commit message: Rework FSP-8 footprint for WS2811 symbol
Parts:
- U1: footprint package:FSOP-8_L3.3-W1.7-P0.80-LS2.9-BL -> package:FSOP-8_3.3x1.7mm_P0.80mm
Changed lines of the file:
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@@
 		)
 	)
-	(footprint "package:FSOP-8_L3.3-W1.7-P0.80-LS2.9-BL"
+	(footprint "package:FSOP-8_3.3x1.7mm_P0.80mm"
 		(layer "B.Cu")
 		(at 163.5 83.5 180)
@@
 			)
 		)
-		(property "Footprint" "package:FSOP-8_L3.3-W1.7-P0.80-LS2.9-BL"
+		(property "Footprint" "package:FSOP-8_3.3x1.7mm_P0.80mm"
 			(at 0 0 90)
 			(layer "B.Fab")
@@
 		)
 		(property "LCSC Part" "C5446692"
-			(at 0 0 0)
+			(at 0 0 180)
 			(unlocked yes)
 			(layer "B.Fab")
@@
 			)
 		)
+		(property ki_fp_filters "*SOP*3.3x1.7mm*P0.80mm*")
 		(sheetname "Root")
 		(sheetfile "esp-doorbell-dev.kicad_sch")
 		(attr smd)
 		(fp_line
-			(start -0.8 1.63)
-			(end 0.8 1.63)
-			(stroke
-				(width 0.12)
-				(type solid)
-			)
-			(layer "B.SilkS")
-		)
-		(fp_line
-			(start -0.8 -1.62)
-			(end 0.8 -1.62)
+			(start -0.8 1.75)
+			(end 0.8 1.75)
+			(stroke
+				(width 0.12)
+				(type solid)
+			)
+			(layer "B.SilkS")
+		)
+		(fp_line
+			(start -0.8 -1.75)
+			(end 0.8 -1.75)
 			(stroke
 				(width 0.12)
@@
 			(layer "B.SilkS")
 		)
-		(fp_circle
-			(center -1.27 1.78)
-			(end -1.27 1.65)
-			(stroke
-				(width 0.25)
-				(type solid)
+		(fp_rect
+			(start -2.05 1.9)
+			(end 2.05 -1.9)
+			(stroke
+				(width 0.05)
+				(type default)
 			)
 			(fill none)
-			(layer "Cmts.User")
+			(layer "B.CrtYd")
 		)
 		(fp_rect
-			(start -1.8 1.63)
-			(end 1.8 -1.62)
-			(stroke
-				(width 0.05)
+			(start -0.85 1.65)
+			(end 0.85 -1.65)
+			(stroke
+				(width 0.1)
 				(type default)
-			)
-			(fill none)
-			(layer "B.CrtYd")
-		)
-		(fp_circle
-			(center -1.43 1.62)
-			(end -1.43 1.59)
-			(stroke
-				(width 0.06)
-				(type solid)
 			)
 			(fill none)
@@
 		(layer "B.Cu")
 		(at 162.55 101.75 -90)
-		(descr "JST XH series connector, S6B-XH-A-1 (http://www.jst-mfg.com/product/pdf/eng/eXH.pdf), generated with kicad-footprint-generator")
+		(descr "JST XH series connector, S6B-XH-2AW")
 		(tags "connector JST XH horizontal")
 		(property "Reference" "J1"
@@
 			(pintype "passive")
 		)
-		(model "${KIPRJMOD}/libraries/lcsc.3dshapes/CONN-TH_XH2.50-WI-6P.wrl"
+		(model "${KIPRJMOD}/libraries/lcsc.3dshapes/CONN-TH_6P-P2.50_DEALON_XH-W-6A.wrl"
 			(offset
-				(xyz 0 -4.6 -2.4)
+				(xyz 6.25 -3.6 3)
 			)
 			(scale
-				(xyz 0.985 1 1)
+				(xyz 1 1.08 1)
 			)
 			(rotate

Commit message: Update URL to pcb.smkent.net on remaining boards
Other:
- board text added: "pcb.smkent.net"
- board text removed: "github.com/smkent/pcb"
Changed lines of the file:
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@@
 		)
 	)
-	(gr_text "github.com/smkent/pcb"
+	(gr_text "pcb.smkent.net"
 		(at 160 157.5 0)
 		(layer "B.SilkS")
 		(effects
 			(font
-				(size 0.8 0.8)
-				(thickness 0.16)
+				(size 1 1)
+				(thickness 0.2)
 				(bold yes)
 			)
