File: pcb/stackable3/ir-trx/ir-trx.kicad_pcb (KiCad board)
At the start: 2 copper layers, 32 x 32 mm, 47 parts, among them J1 PJ-327U, Q1 G2N7002X, Q2 DMP1045U, Q3 DMG6968U, SW1 SW_SPDT_MountingPin, U1 DY-IRMHA384

Commit message: Replace discrete resistor footprints with built-ins on stackable3 boards
Parts:
- R14: footprint discrete:R_0603_1608Metric -> Resistor_SMD:R_0603_1608Metric
